File: 2019_Rev1_Sensor_Board/2019_Rev1_Sensor_Board.kicad_pcb (KiCad board)
At the start: 2 copper layers, 124.6 x 91.3 mm, 24 parts, among them U1 Tive Header, U2 AP1059, U4 AP1059

Commit message: worked on SRA board review
Routing:
- net +5V: track 107.0 -> 54.1 mm
- net Bit7: track 62.4 -> 86.2 mm
Changed lines of the file:
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@@
     (thickness 1.6)
     (drawings 19)
-    (tracks 215)
+    (tracks 214)
     (zones 0)
     (modules 24)
@@
   (segment (start 176.784 99.822) (end 152.654 99.822) (width 0.381) (layer F.Cu) (net 2))
   (via (at 152.654 99.822) (size 0.8) (drill 0.4) (layers F.Cu B.Cu) (net 2))
-  (segment (start 152.654 99.822) (end 99.695 99.822) (width 0.381) (layer B.Cu) (net 2))
   (segment (start 115.076 58.434) (end 115.062 58.42) (width 0.381) (layer F.Cu) (net 3))
   (segment (start 115.076 62.865) (end 115.076 58.434) (width 0.381) (layer F.Cu) (net 3))
@@
   (segment (start 163.749001 98.217001) (end 163.749001 98.552) (width 0.381) (layer B.Cu) (net 68))
   (segment (start 163.749001 98.552) (end 163.749001 107.145001) (width 0.381) (layer B.Cu) (net 68))
-  (segment (start 161.209001 99.233001) (end 161.209001 107.145001) (width 0.381) (layer B.Cu) (net 69))
-  (segment (start 128.778 59.49763) (end 128.524 59.75163) (width 0.381) (layer B.Cu) (net 69))
   (segment (start 128.778 58.42) (end 128.778 59.49763) (width 0.381) (layer B.Cu) (net 69))
-  (segment (start 128.524 59.75163) (end 128.524 63.754) (width 0.381) (layer B.Cu) (net 69))
-  (segment (start 161.209001 96.439001) (end 161.209001 99.233001) (width 0.381) (layer B.Cu) (net 69))
-  (segment (start 128.524 63.754) (end 161.209001 96.439001) (width 0.381) (layer B.Cu) (net 69))
+  (segment (start 130.4036 105.2068) (end 161.209001 105.2068) (width 0.25) (layer B.Cu) (net 69))
+  (segment (start 128.778 103.5812) (end 130.4036 105.2068) (width 0.25) (layer B.Cu) (net 69))
+  (segment (start 161.209001 99.233001) (end 161.209001 105.2068) (width 0.381) (layer B.Cu) (net 69))
+  (segment (start 128.778 59.49763) (end 128.778 103.5812) (width 0.25) (layer B.Cu) (net 69))
+  (segment (start 161.209001 105.2068) (end 161.209001 107.145001) (width 0.381) (layer B.Cu) (net 69))
   (segment (start 159.429 65.745002) (end 158.669001 66.505001) (width 0.381) (layer F.Cu) (net 70))
   (segment (start 159.819502 65.3545) (end 159.429 65.745002) (width 0.381) (layer F.Cu) (net 70))
