File: 2019_Rev1_Sensor_Board/2019_Rev1_Sensor_Board.sch (KiCad schematic (older format))
At the start: 30 parts, among them U1 Tive Header, U2 AP1059, U4 AP1059

Commit message: worked on SRA board review
Parts:
- added Conn?: Molex_SL_04, symbol MRDT_Connectors:Molex_SL_04
- added D10, D11, D7, D8, D9: LED, Diode_SMD:D_0603_1608Metric_Pad1.05x0.95mm_HandSolder, symbol Device:LED
- added R10, R11, R12, R13, R8, R9: 500, Resistor_SMD:R_0603_1608Metric_Pad1.05x0.95mm_HandSolder, symbol Device:R
- gave numbers to parts that had none: 6
- renumbered PWR1 to D3, H1 to L1, H2 to L2
Connections:
- net labels added: AnalogOut, ERROR, Soft_Flag1, Soft_Flag2
- net labels removed: AnalogIn
- wire segments 155 -> 169
Other:
- note added: "BLU"
- note added: "CCD STUFF\n"
- note added: "GREN\n"
- note added: "RED\n"
- note added: "YELO\n"
- note removed: "Power LED"
