File: 2019_Rev1_Sensor_Board/SRASensorBoard_Hardware.kicad_pcb (KiCad board)
At the start: 2 copper layers, 124.6 x 91.3 mm, 24 parts, among them U1 Tive Header, U2 AP1059, U4 AP1059

Commit message: Retraced SRA Board
Parts:
- removed H1, H2: 47u, Inductor_SMD:L_0603_1608Metric_Pad1.05x0.95mm_HandSolder
- removed PWR: LED, Diode_SMD:D_0603_1608Metric_Pad1.05x0.95mm_HandSolder
- added Conn9: Molex_SL_04, MRDT_Connectors:MOLEX_SL_04_Horizontal, F.Cu at (115.1, 58.3)
- added D10: LED, Diode_SMD:D_0603_1608Metric_Pad1.05x0.95mm_HandSolder, F.Cu at (164.3, 81.2)
- added D11: LED, Diode_SMD:D_0603_1608Metric_Pad1.05x0.95mm_HandSolder, F.Cu at (164.4, 84.5)
- added D3: LED, Diode_SMD:D_0603_1608Metric_Pad1.05x0.95mm_HandSolder, F.Cu at (191.3, 72.6)
- added D4: LED, Diode_SMD:D_0603_1608Metric_Pad1.05x0.95mm_HandSolder, F.Cu at (191.3, 70.3)
- added D5: LED, Diode_SMD:D_0603_1608Metric_Pad1.05x0.95mm_HandSolder, F.Cu at (152.7, 76.8)
- added D6: LED, Diode_SMD:D_0603_1608Metric_Pad1.05x0.95mm_HandSolder, F.Cu at (152.7, 82.7)
- added D7: LED, Diode_SMD:D_0603_1608Metric_Pad1.05x0.95mm_HandSolder, F.Cu at (152.8, 79.8)
- added D8: LED, Diode_SMD:D_0603_1608Metric_Pad1.05x0.95mm_HandSolder, F.Cu at (152.8, 85.6)
- added D9: LED, Diode_SMD:D_0603_1608Metric_Pad1.05x0.95mm_HandSolder, F.Cu at (164.3, 78.0)
- added G***: LOGO, MRDT_Silkscreens:MRDT_Logo_20mm, F.Cu at (198.1, 123.8)
- added G***: LOGO, MRDT_Silkscreens:MRDT_Retro_Logo_34mmX21.5mm, F.Cu at (105.0, 124.8)
- added L1: 47u, Inductor_SMD:L_0603_1608Metric_Pad1.05x0.95mm_HandSolder, F.Cu at (197.7, 81.5)
- added L2: 47u, Inductor_SMD:L_0603_1608Metric_Pad1.05x0.95mm_HandSolder, F.Cu at (185.7, 81.5)
- added R10: 500, Resistor_SMD:R_0603_1608Metric_Pad1.05x0.95mm_HandSolder, F.Cu at (167.9, 78.0)
- added R11: 500, Resistor_SMD:R_0603_1608Metric_Pad1.05x0.95mm_HandSolder, F.Cu at (167.8, 81.2)
- added R12: 500, Resistor_SMD:R_0603_1608Metric_Pad1.05x0.95mm_HandSolder, F.Cu at (167.9, 84.5)
- added R13: 500, Resistor_SMD:R_0603_1608Metric_Pad1.05x0.95mm_HandSolder, B.Cu at (158.9, 58.3)
- added R5: 500, Resistor_SMD:R_0603_1608Metric_Pad1.05x0.95mm_HandSolder, F.Cu at (187.7, 70.3)
- added R6: 500, Resistor_SMD:R_0603_1608Metric_Pad1.05x0.95mm_HandSolder, F.Cu at (149.1, 76.8)
- added R7: 500, Resistor_SMD:R_0603_1608Metric_Pad1.05x0.95mm_HandSolder, F.Cu at (149.2, 82.7)
- added R8: 500, Resistor_SMD:R_0603_1608Metric_Pad1.05x0.95mm_HandSolder, F.Cu at (149.2, 79.8)
- added R9: 500, Resistor_SMD:R_0603_1608Metric_Pad1.05x0.95mm_HandSolder, F.Cu at (149.3, 85.6)
- R2, R3, R4: moved to B.Cu
- moved Conn5 44.4 mm to (201.5, 58.2), turned to 0 degrees
- moved Conn1 33.1 mm to (186.3, 94.7), turned to 180 degrees
- moved R2 21.3 mm to (98.4, 61.0), turned to 0 degrees
- moved Conn2 20.2 mm to (100.6, 58.3), turned to 0 degrees
- moved Conn4 19.0 mm to (99.4, 76.7)
- moved R4 19.0 mm to (103.9, 74.5)
- moved R1 14.8 mm to (187.7, 72.7), turned to 0 degrees
- moved R3 11.5 mm to (127.4, 61.5)
- moved Conn3 10.7 mm to (128.3, 58.3)
- moved Conn7 8.89 mm to (146.6, 58.3)
- moved Conn6 7.11 mm to (163.6, 58.3)
- moved C4 5.19 mm to (188.8, 85.4), turned to 180 degrees
- moved Conn8 4.57 mm to (180.6, 58.3)
- moved D2 3.94 mm to (186.6, 78.0)
- moved C2 3.28 mm to (191.3, 78.0)
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Connections:
- net AnalogIn renamed AnalogOut
- C3 pad 1: +3V3 -> GND
- C3 pad 2: GND -> +3V3
- C4 pad 1: +5V -> GND
- C4 pad 2: GND -> +5V
- Conn6 pad 1: TOGGLE -> Net-(Conn6-Pad1)
- R1 pad 1: +5V -> +3V3
- U1 pad PB5: Net-(U1-PadPB5) -> Soil_Sck
- U1 pad PC4: Net-(U1-PadPC4) -> Methane_Vout
- U1 pad PE0: Net-(U1-PadPE0) -> Master_CLOCK
- U1 pad PE3: Net-(U1-PadPE3) -> Shift_Gate
- U1 pad PE4: Methane_Vout -> ICG
- U1 pad PF1: Net-(U1-PadPF1) -> SDATA
- U1 pad PF2: Net-(U1-PadPF2) -> SCLK
- U1 pad PF3: Soil_Sck -> CS
- U1 pad PG1: ICG -> Net-(U1-PadPG1)
- U1 pad PH0: Shift_Gate -> Net-(U1-PadPH0)
- U1 pad PN4: Net-(U1-PadPN4) -> ERROR
- U1 pad PN5: Net-(U1-PadPN5) -> Soft_Flag1
- U1 pad PP4: Net-(U1-PadPP4) -> Soft_Flag2
- U1 pad PQ0: Master_CLOCK -> Net-(U1-PadPQ0)
- U1 pad PQ1: CS -> Net-(U1-PadPQ1)
- U1 pad PQ2: SDATA -> Net-(U1-PadPQ2)
- U1 pad PQ3: SCLK -> Net-(U1-PadPQ3)
Routing:
- net +5V: track 54.1 -> 200.8 mm
- net Master_CLOCK: track 28.3 -> 163.7 mm, vias 0 -> 1
- net ICG: track 58.9 -> 168.7 mm
- net Shift_Gate: track 53.7 -> 160.1 mm, vias 0 -> 2
- net Soil_Sck: track 18.3 -> 99.4 mm
- net Methane_Vout: track 30.6 -> 104.7 mm, vias 0 -> 1
- net Soil_Data: track 23.2 -> 71.1 mm, vias 0 -> 1
- net Atm_Dout: track 17.9 -> 64.2 mm, vias 0 -> 2
- net ERROR: track 0.00 -> 38.2 mm
- net +3V3: track 32.8 -> 70.8 mm, vias 0 -> 1
- net SCLK: track 0.00 -> 36.1 mm, vias 0 -> 1
- net Soft_Flag1: track 0.00 -> 35.9 mm
- net SDATA: track 0.00 -> 35.8 mm, vias 0 -> 1
- net Bit5: track 95.7 -> 130.4 mm
- net Soft_Flag2: track 0.00 -> 33.7 mm
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Other:
- board text added: "+3.3V"
- board text added: "+5V"
- board text added: "1 2 3 4"
- board text added: "ATM LED"
- board text added: "ATM Sensor"
- board text added: "Austin Christman, Austin Hill, Kamran Winschel"
- board text added: "CCD"
- board text added: "CCD Bits 1-7"
- board text added: "CCD Bits 8-14"
- board text added: "Debug LEDS"
- board text added: "Error"
- board text added: "Mars Rover Design Team"
- board text added: "Missouri S&T"
- board text added: "Mthn LED"
- board text added: "PWR LEDS"
- board text added: "Science Research and Analysis"
- board text added: "Sensor LEDS"
- board text added: "Sft Flg1"
- board text added: "Sft Flg2"
- board text added: "Soil LED"
- board text added: "Soil Sensor"
- board text added: "UV LED"

Commit message: revised more on the pcb for SRA
Parts:
- moved D10 1.27 mm to (164.3, 79.9)
- moved R11 1.27 mm to (167.8, 79.9)
- moved D11 1.27 mm to (164.4, 83.2)
- moved D9 1.27 mm to (164.3, 76.7)
- moved R10 1.27 mm to (167.9, 76.7)
- moved R12 1.27 mm to (167.9, 83.2)
Routing:
- net +3V3: track 70.8 -> 9.24 mm, vias 1 -> 4
- net Bit3: track 98.2 -> 102.0 mm
- net Net-(C1-Pad1): track 61.8 -> 64.3 mm, vias 2 -> 1
- net ERROR: track 38.2 -> 39.6 mm
- net Soft_Flag1: track 35.9 -> 37.2 mm
- net Soft_Flag2: track 33.7 -> 35.0 mm
- net AnalogOut: track 37.3 -> 38.4 mm
- net SCLK: track 36.1 -> 35.0 mm
- net Bit14: track 24.5 -> 25.4 mm
Other:
- board text added: "+3V3"
- board text added: "2 1"
- board text added: "3 2 1"
- board text added: "4 3 2 1"
- board text added: "5 4 3 2 1"
- board text added: "8 7 6 5 4 3 2 1"
- board text added: "AO"
- board text added: "ATM Sensor AM2302"
- board text added: "Atm_Dout"
- board text added: "Bit0"
- board text added: "Bit1"
- board text added: "Bit10"
- board text added: "Bit11"
- board text added: "Bit12"
- board text added: "Bit13"
- board text added: "Bit14"
- board text added: "Bit2"
- board text added: "Bit3"
- board text added: "Bit4"
- board text added: "Bit5"
- board text added: "Bit6"
- board text added: "Bit7"
- board text added: "Bit8"
- board text added: "Bit9"
- board text added: "CS"
- board text added: "GND"
- board text added: "ICG"
- board text added: "MTHN Sensor MQ-4"
- board text added: "Mstr CLK"
- board text added: "Mthn Vout"
- board text added: "SCLK"
- board text added: "SDATA"
- board text added: "SRA Board Rev1 2019 Mars Rover Design Team Missouri S&T Austin Christman, Austin Hill, Kamran Winschel"
- board text added: "SW Error"
- board text added: "SW Flg1"
- board text added: "SW Flg2"
- board text added: "Shft Gate"
- board text added: "Soil T/M SHT-10"
- board text added: "Soil_Data"
- board text added: "Soil_Sck"
- board text added: "UVTOG"
- board text removed: "1 2 3 4"
- board text removed: "ATM Sensor"
- board text removed: "Austin Christman, Austin Hill, Kamran Winschel"
- board text removed: "Error"
- board text removed: "Mars Rover Design Team"
- board text removed: "Missouri S&T"
- board text removed: "Science Research and Analysis"
- board text removed: "Sft Flg1"
- board text removed: "Sft Flg2"
- board text removed: "Soil Sensor"

Commit message: More Updates
Fixed small traceing errors, folder managment, etc.
Parts:
- moved D3 2.54 mm to (191.3, 70.1)
- moved D4 2.54 mm to (191.3, 67.7)
- moved R5 2.54 mm to (187.7, 67.8)
- moved R1 2.54 mm to (187.7, 70.1)
Routing:
- net Net-(C1-Pad1): track 64.3 -> 74.5 mm
- net +5V: track 200.7 -> 203.2 mm
Other:
- board text added: "SRA Sensor Board Hardware Rev1 2019 Mars Rover Design Team Missouri S&T Austin Christman, Austin Hill, Kamran Winschel"
- board text removed: "SRA Board Rev1 2019 Mars Rover Design Team Missouri S&T Austin Christman, Austin Hill, Kamran Winschel"

Commit message: Rev1
Parts:
- removed D1, D2: D_Schottky, Diode_SMD:D_0603_1608Metric_Pad1.05x0.95mm_HandSolder
- removed L1, L2: 47u, Inductor_SMD:L_0603_1608Metric_Pad1.05x0.95mm_HandSolder
- removed U4: AP1059, Package_SO:SOIC-8_3.9x4.9mm_P1.27mm
- added G***: LOGO, SRA_Hardware:Austin_Hill_Sig_22mmx9.3mm, F.Cu at (169.8, 132.6)
- added U3: OKI, MRDT_Devices:OKI_Horizontal, F.Cu at (193.5, 73.4)
- U2: value AP1059 -> OKI; footprint Package_SO:SOIC-8_3.9x4.9mm_P1.27mm -> MRDT_Devices:OKI_Horizontal
- moved C4 19.1 mm to (190.9, 66.4), turned to 270 degrees
- moved D4 16.3 mm to (184.9, 82.7), turned to 90 degrees
- moved D3 15.4 mm to (182.5, 82.7), turned to 90 degrees
- moved C1 14.9 mm to (190.9, 69.8), turned to 90 degrees
- moved R5 11.7 mm to (184.8, 79.1), turned to 270 degrees
- moved C3 10.5 mm to (190.8, 82.5), turned to 90 degrees
- moved R1 10.4 mm to (182.5, 79.1), turned to 270 degrees
- moved U2 10.3 mm to (193.5, 85.9), turned to 90 degrees
- moved Conn1 1.61 mm to (186.9, 93.2)
- moved C2 1.21 mm to (190.8, 79.1), turned to 270 degrees
Connections:
- net ERROR renamed SW_ERROR
- net Soft_Flag1 renamed SW_Flag1
- net Soft_Flag2 renamed SW_Flag2
- net TOGGLE renamed UV_TOGGLE
- C2 pad 1: Net-(C1-Pad1) -> +5V
- C3 pad 1: GND -> Net-(C1-Pad1)
- C3 pad 2: +3V3 -> GND
- C4 pad 1: GND -> +3V3
- C4 pad 2: +5V -> GND
- U2 pad 2: Net-(D1-Pad1) -> GND
- U2 pad 3: +3V3 -> +5V
Routing:
- net Net-(C1-Pad1): track 74.5 -> 52.9 mm, vias 1 -> 0
- net Net-(D1-Pad1): track 5.30 -> 0.00 mm
- net Net-(D2-Pad1): track 5.27 -> 0.00 mm
- net +5V: track 203.2 -> 207.4 mm
- net +3V3: track 9.24 -> 11.9 mm, vias 4 -> 6
- net UV_TOGGLE: track 28.8 -> 29.6 mm
Other:
- board text added: "PWR"
- board text added: "SRA Sensor Board Hardware, Rev1 Mars Rover Design Team Missouri S&T, 2019 Austin Christman, Austin Hill, Kamran Winschel"
- board text removed: "PWR LEDS"
- board text removed: "SRA Sensor Board Hardware Rev1 2019 Mars Rover Design Team Missouri S&T Austin Christman, Austin Hill, Kamran Winschel"

Commit message: Worked on files
Parts:
- added G***: LOGO, SRA_Hardware:Austin_Christman_Sig_22mmx8.3mm, F.Cu at (137.0, 132.0)
- moved G*** 3.96 mm to (165.9, 133.0)
- moved C1 0.37 mm to (190.9, 70.2)
- moved D8 0.34 mm to (153.1, 85.6)
- moved D6 0.30 mm to (153.0, 82.7)
- moved D7 0.29 mm to (153.0, 79.8)
- moved C3 0.28 mm to (190.8, 82.8)
- moved D5 0.27 mm to (153.0, 76.8)
- moved D4 0.22 mm to (184.9, 82.9)
- moved D3 0.21 mm to (182.5, 82.9)
- moved R11 0.21 mm to (168.0, 79.9)
- moved C2 0.14 mm to (190.8, 79.0)
- moved R10 0.14 mm to (168.0, 76.7)
- moved R12 0.13 mm to (168.0, 83.2)
- moved C4 0.13 mm to (190.9, 66.3)
- moved R8 0.10 mm to (149.1, 79.8)
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Connections:
- U1 pad PA7: AnalogOut -> Net-(U1-PadPA7)
- U1 pad PC4: Methane_Vout -> Net-(U1-PadPC4)
- U1 pad PD0: Soil_Data -> Net-(U1-PadPD0)
- U1 pad PD1: Net-(U1-PadPD1) -> AnalogOut
- U1 pad PE1: Net-(U1-PadPE1) -> ICG
- U1 pad PE2: Net-(U1-PadPE2) -> Methane_Vout
- U1 pad PE4: ICG -> Net-(U1-PadPE4)
- U1 pad PE5: Net-(U1-PadPE5) -> Soil_Data
Routing:
- net AnalogOut: track 38.4 -> 106.5 mm, vias 1 -> 2
- net Soil_Data: track 71.1 -> 116.7 mm, vias 1 -> 2
- net +5V: track 207.4 -> 196.4 mm
- net Methane_Vout: track 104.6 -> 94.7 mm
- net GND: track 4.77 -> 9.62 mm, vias 0 -> 1
- net ICG: track 168.3 -> 164.9 mm, vias 1 -> 2
- net +3V3: track 11.9 -> 10.3 mm, vias 6 -> 4
- net Net-(C1-Pad1): track 52.9 -> 53.8 mm
Other:
- board text added: "ATM T/H AM2302"
- board text added: "CCD TCD1304DG"
- board text added: "Soil T/H SHT-10"
- board text removed: "ATM Sensor AM2302"
- board text removed: "Soil T/M SHT-10"
