File: 2019_Rev1_Sensor_Board/SRASensorBoard_Hardware.sch (KiCad schematic (older format))
At the start: 42 parts, among them U1 Tive Header, U2 AP1059, U4 AP1059

Commit message: Retraced SRA Board
Parts:
- Conn9: renamed from Conn?; footprint (none) -> MRDT_Connectors:MOLEX_SL_04_Horizontal
Connections:
- wire segments 169 -> 172

Commit message: revised more on the pcb for SRA
Connections:
- net labels added: SW_ERROR, SW_Flag1, SW_Flag2, UV-TOGGLE, UV_TOGGLE
- net labels removed: ERROR, Soft_Flag1, Soft_Flag2, TOGGLE
- wire segments 172 -> 181

Commit message: More Updates
Fixed small traceing errors, folder managment, etc.
Connections:
- wire segments 181 -> 182
Other:
- note added: "12/19/18"
- note added: "Number 1"
- note added: "SRA Sensor Board Hardware"
Changed lines of the file:
@@
 L power:GND #PWR0101
 U 1 1 5BCB97F5
-P 3250 2650
-F 0 "#PWR0101" H 3250 2400 50  0001 C CNN
-F 1 "GND" H 3255 2477 50  0000 C CNN
-F 2 "" H 3250 2650 50  0001 C CNN
-F 3 "" H 3250 2650 50  0001 C CNN
-	1    3250 2650
+P 3250 2750
+F 0 "#PWR0101" H 3250 2500 50  0001 C CNN
+F 1 "GND" H 3255 2577 50  0000 C CNN
+F 2 "" H 3250 2750 50  0001 C CNN
+F 3 "" H 3250 2750 50  0001 C CNN
+	1    3250 2750
 	-1   0    0    -1
 $EndComp
@@
 L power:+3.3V #PWR01
 U 1 1 5BE81B23
-P 3000 1900
-F 0 "#PWR01" H 3000 1750 50  0001 C CNN
-F 1 "+3.3V" V 3100 1950 50  0000 C CNN
-F 2 "" H 3000 1900 50  0001 C CNN
-F 3 "" H 3000 1900 50  0001 C CNN
-	1    3000 1900
-	0    1    1    0
+P 3100 1900
+F 0 "#PWR01" H 3100 1750 50  0001 C CNN
+F 1 "+3.3V" H 3100 1850 50  0000 C CNN
+F 2 "" H 3100 1900 50  0001 C CNN
+F 3 "" H 3100 1900 50  0001 C CNN
+	1    3100 1900
+	1    0    0    -1
 $EndComp
 $Comp
@@
 L power:+5V #PWR02
 U 1 1 5BED3911
-P 3050 2950
-F 0 "#PWR02" H 3050 2800 50  0001 C CNN
-F 1 "+5V" V 3150 3000 50  0000 C CNN
-F 2 "" H 3050 2950 50  0001 C CNN
-F 3 "" H 3050 2950 50  0001 C CNN
-	1    3050 2950
-	0    1    1    0
+P 3100 2950
+F 0 "#PWR02" H 3100 2800 50  0001 C CNN
+F 1 "+5V" H 3100 2900 50  0000 C CNN
+F 2 "" H 3100 2950 50  0001 C CNN
+F 3 "" H 3100 2950 50  0001 C CNN
+	1    3100 2950
+	1    0    0    -1
 $EndComp
 $Comp
@@
 Connection ~ 2900 1900
 Wire Wire Line
-	2900 1900 3000 1900
-Wire Wire Line
 	3250 1550 3250 2250
 Connection ~ 3250 2250
@@
 Connection ~ 2950 2950
 Wire Wire Line
-	2950 2950 3050 2950
-Wire Wire Line
 	2400 2450 2300 2450
 Wire Wire Line
@@
 Wire Wire Line
 	10850 5900 10850 5950
+Wire Wire Line
+	2900 1900 3100 1900
+Wire Wire Line
+	3250 2750 3250 2650
+Wire Wire Line
+	2950 2950 3100 2950
+Text Notes 8140 7645 0    59   ~ 0
+12/19/18
+Text Notes 7350 7510 0    79   ~ 0
+SRA Sensor Board Hardware
+Text Notes 10580 7645 0    59   ~ 0
+Number 1
 $EndSCHEMATC

Commit message: Rev1
Parts:
- removed D1, D2: D_Schottky, Diode_SMD:D_0603_1608Metric_Pad1.05x0.95mm_HandSolder, symbol Device:D_Schottky
- removed L1, L2: 47u, Inductor_SMD:L_0603_1608Metric_Pad1.05x0.95mm_HandSolder, symbol pspice:INDUCTOR
- removed U2, U4: AP1059, Package_SO:SOIC-8_3.9x4.9mm_P1.27mm, symbol MRDT_ICs:AP1059
- added U2, U3: OKI, MRDT_Devices:OKI_Horizontal, symbol MRDT_Devices:OKI
Connections:
- net labels removed: UV-TOGGLE
- wire segments 182 -> 152
Other:
- note added: "CCD Breakout\n"
- note removed: "CCD STUFF\n"

Commit message: Worked on files
Other:
- note added: "SPI 1"
- note added: "SPI 1\n"
- note added: "SPI 3"
