File: SRASensorBoard_Hardware/_autosave-SRASensorBoard_Hardware.kicad_pcb (KiCad board)
At the start: 2 copper layers, 124.6 x 91.3 mm, 42 parts, among them U1 Tive Header, U2 OKI, U3 OKI

Commit message: PR ready
Routing:
- net GND: track 9.62 -> 33.2 mm, vias 1 -> 7
- net Soil_Data: track 116.7 -> 123.6 mm
- net +3V3: track 10.3 -> 6.11 mm, vias 4 -> 1
Other:
- board text added: "+12V"
- board text added: "SRA Sensor Board Hardware, Rev1 Mars Rover Design Team Missouri S&T, 2019 Austin Christman, Austin Hill"
- board text removed: "SRA Sensor Board Hardware, Rev1 Mars Rover Design Team Missouri S&T, 2019 Austin Christman, Austin Hill, Kamran Winschel"
