File: SRASensorBoard_Hardware/SRASensorBoard_Hardware.kicad_pcb (KiCad board)
At the start: 2 copper layers, 124.6 x 91.3 mm, 42 parts, among them U1 Tive Header, U2 OKI, U3 OKI

Commit message: updated schematic
Parts:
- removed Conn7, Conn8: Molex_SL_08, MRDT_Connectors:MOLEX_SL_08_Horizontal
- removed Conn9: Molex_SL_04, MRDT_Connectors:MOLEX_SL_04_Horizontal
- added D1: LED, Diode_SMD:D_0603_1608Metric_Pad1.05x0.95mm_HandSolder, F.Cu at (153.1, 88.4)
- added R14: 500, Resistor_SMD:R_0603_1608Metric_Pad1.05x0.95mm_HandSolder, F.Cu at (149.2, 88.4)
- Conn5: value Molex_SL_05 -> Molex_SL_03; footprint MRDT_Connectors:MOLEX_SL_05_Horizontal -> MRDT_Connectors:MOLEX_SL_03_Horizontal
- moved Conn5 18.6 mm to (182.9, 58.4)
Connections:
- net Master_CLOCK renamed CCD_INT
- Conn5 pad 3: ICG -> GND
- U1 pad PA4: Net-(U1-PadPA4) -> (no net)
- U1 pad PA5: Net-(U1-PadPA5) -> (no net)
- U1 pad PA6: Net-(U1-PadPA6) -> (no net)
- U1 pad PA7: Net-(U1-PadPA7) -> (no net)
- U1 pad PB2: Net-(U1-PadPB2) -> (no net)
- U1 pad PB3: Net-(U1-PadPB3) -> (no net)
- U1 pad PB4: Net-(U1-PadPB4) -> (no net)
- U1 pad PC4: Net-(U1-PadPC4) -> (no net)
- U1 pad PC5: Net-(U1-PadPC5) -> (no net)
- U1 pad PC6: Net-(U1-PadPC6) -> (no net)
- U1 pad PC7: Net-(U1-PadPC7) -> (no net)
- U1 pad PD0: Net-(U1-PadPD0) -> (no net)
- U1 pad PD1: AnalogOut -> (no net)
- U1 pad PD2: Net-(U1-PadPD2) -> (no net)
- U1 pad PD3: Net-(U1-PadPD3) -> (no net)
- U1 pad PD4: Net-(U1-PadPD4) -> (no net)
- U1 pad PD5: Net-(U1-PadPD5) -> (no net)
- U1 pad PD7: Net-(U1-PadPD7) -> (no net)
- U1 pad PE1: ICG -> (no net)
- U1 pad PE3: Shift_Gate -> (no net)
- U1 pad PE4: Net-(U1-PadPE4) -> (no net)
- U1 pad PF1: SDATA -> (no net)
- U1 pad PF2: SCLK -> (no net)
- U1 pad PF3: CS -> (no net)
- U1 pad PG0: Net-(U1-PadPG0) -> (no net)
- U1 pad PG1: Net-(U1-PadPG1) -> (no net)
- U1 pad PH0: Net-(U1-PadPH0) -> (no net)
- U1 pad PH1: Net-(U1-PadPH1) -> (no net)
- U1 pad PH2: Net-(U1-PadPH2) -> (no net)
- U1 pad PH3: Net-(U1-PadPH3) -> (no net)
- U1 pad PK0: Bit7 -> (no net)
- U1 pad PK1: Bit8 -> (no net)
- U1 pad PK2: Bit9 -> (no net)
- U1 pad PK3: Bit10 -> (no net)
- U1 pad PK4: Bit11 -> (no net)
- U1 pad PK5: Bit12 -> (no net)
- U1 pad PK6: Bit13 -> (no net)
- U1 pad PK7: Bit14 -> (no net)
- U1 pad PL0: Net-(U1-PadPL0) -> (no net)
- U1 pad PL1: Net-(U1-PadPL1) -> (no net)
- U1 pad PL2: Net-(U1-PadPL2) -> (no net)
- U1 pad PL3: Net-(U1-PadPL3) -> (no net)
- U1 pad PL4: Net-(U1-PadPL4) -> (no net)
- U1 pad PL5: Net-(U1-PadPL5) -> (no net)
- U1 pad PM0: Bit0 -> (no net)
- U1 pad PM1: Bit1 -> (no net)
- U1 pad PM2: Bit2 -> (no net)
- U1 pad PM3: Bit3 -> (no net)
- U1 pad PM4: Bit4 -> (no net)
- U1 pad PM5: Bit5 -> (no net)
- U1 pad PM6: Bit6 -> (no net)
- U1 pad PM7: Net-(U1-PadPM7) -> (no net)
- U1 pad PN3: Net-(U1-PadPN3) -> (no net)
- U1 pad PP0: Net-(U1-PadPP0) -> (no net)
- U1 pad PP1: Net-(U1-PadPP1) -> (no net)
- U1 pad PP2: Net-(U1-PadPP2) -> (no net)
- U1 pad PP3: Net-(U1-PadPP3) -> (no net)
- U1 pad PQ0: Net-(U1-PadPQ0) -> (no net)
- U1 pad PQ1: Net-(U1-PadPQ1) -> (no net)
- U1 pad PQ2: Net-(U1-PadPQ2) -> (no net)
- U1 pad PQ3: Net-(U1-PadPQ3) -> (no net)
Routing:
- net ICG: track 164.9 -> 0.00 mm, vias 2 -> 0
- net Shift_Gate: track 159.9 -> 0.00 mm, vias 2 -> 0
- net Bit5: track 130.4 -> 0.00 mm, vias 1 -> 0
- net Bit4: track 129.4 -> 0.00 mm, vias 1 -> 0
- net AnalogOut: track 106.0 -> 0.00 mm, vias 2 -> 0
- net Bit3: track 102.0 -> 0.00 mm, vias 2 -> 0
- net Bit10: track 77.5 -> 0.00 mm
- net Bit9: track 74.9 -> 0.00 mm
- net Bit8: track 72.3 -> 0.00 mm
- net Bit7: track 69.7 -> 0.00 mm
- net SDATA: track 35.8 -> 0.00 mm, vias 1 -> 0
- net SCLK: track 35.0 -> 0.00 mm, vias 1 -> 0
- net CS: track 30.3 -> 0.00 mm
- net Bit14: track 25.4 -> 0.00 mm
- net Bit13: track 23.9 -> 0.00 mm
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Other:
- board text added: "CCD LED"
- board text added: "CCD_INT"
- board text added: "CCD_TIVA"
- board text removed: "5 4 3 2 1"
- board text removed: "8 7 6 5 4 3 2 1"
- board text removed: "AO"
- board text removed: "Bit0"
- board text removed: "Bit1"
- board text removed: "Bit10"
- board text removed: "Bit11"
- board text removed: "Bit12"
- board text removed: "Bit13"
- board text removed: "Bit14"
- board text removed: "Bit2"
- board text removed: "Bit3"
- board text removed: "Bit4"
- board text removed: "Bit5"
- board text removed: "Bit6"
- board text removed: "Bit7"
- board text removed: "Bit8"
- board text removed: "Bit9"
- board text removed: "CCD"
- board text removed: "CCD Bits 1-7"
- board text removed: "CCD Bits 8-14"
- board text removed: "CCD TCD1304DG"
- board text removed: "CS"
- board text removed: "ICG"
- board text removed: "Mstr CLK"
- board text removed: "SCLK"
- board text removed: "SDATA"
- board text removed: "Shft Gate"
