File: SRASensorBoard_Hardware/SRASensorBoard_Hardware.sch (KiCad schematic (older format))
At the start: 38 parts, among them U1 Tive Header, U2 OKI, U3 OKI

Commit message: PR ready
Other:
- note added: "A1"
- note added: "A14"
- note removed: "SPI 1"
- note removed: "SPI 1\n"
- moved on the sheet: C1, C2, C3, C4, Conn1A, Conn1B
Changed lines of the file:
@@
 L MRDT_Connectors:AndersonPP Conn1
 U 1 1 5BCC6BDC
-P 1500 2650
-F 0 "Conn1" H 1600 2600 60  0000 C CNN
-F 1 "AndersonPP" H 1550 3250 60  0001 C CNN
-F 2 "MRDT_Connectors:Anderson_2_Horisontal_Side_by_Side" H 1350 2100 60  0001 C CNN
-F 3 "" H 1350 2100 60  0001 C CNN
-	1    1500 2650
+P 1500 2300
+F 0 "Conn1" H 1600 2250 60  0000 C CNN
+F 1 "AndersonPP" H 1550 2900 60  0001 C CNN
+F 2 "MRDT_Connectors:Anderson_2_Horisontal_Side_by_Side" H 1350 1750 60  0001 C CNN
+F 3 "" H 1350 1750 60  0001 C CNN
+	1    1500 2300
 	1    0    0    -1
 $EndComp
@@
 L Device:C_Small C3
 U 1 1 5BF3ACAB
-P 2150 2400
-F 0 "C3" H 2200 2450 50  0000 L CNN
-F 1 "10u" H 2200 2350 50  0000 L CNN
-F 2 "Capacitor_SMD:C_0603_1608Metric_Pad1.05x0.95mm_HandSolder" H 2150 2400 50  0001 C CNN
-F 3 "~" H 2150 2400 50  0001 C CNN
-	1    2150 2400
+P 2150 2050
+F 0 "C3" H 2200 2100 50  0000 L CNN
+F 1 "10u" H 2200 2000 50  0000 L CNN
+F 2 "Capacitor_SMD:C_0603_1608Metric_Pad1.05x0.95mm_HandSolder" H 2150 2050 50  0001 C CNN
+F 3 "~" H 2150 2050 50  0001 C CNN
+	1    2150 2050
 	1    0    0    -1
 $EndComp
@@
 L Device:C_Small C4
 U 1 1 5BF44706
-P 3000 2400
-F 0 "C4" H 2850 2450 50  0000 L CNN
-F 1 "10u" H 2850 2350 50  0000 L CNN
-F 2 "Capacitor_SMD:C_0603_1608Metric_Pad1.05x0.95mm_HandSolder" H 3000 2400 50  0001 C CNN
-F 3 "~" H 3000 2400 50  0001 C CNN
-	1    3000 2400
+P 3000 2050
+F 0 "C4" H 2850 2100 50  0000 L CNN
+F 1 "10u" H 2850 2000 50  0000 L CNN
+F 2 "Capacitor_SMD:C_0603_1608Metric_Pad1.05x0.95mm_HandSolder" H 3000 2050 50  0001 C CNN
+F 3 "~" H 3000 2050 50  0001 C CNN
+	1    3000 2050
 	1    0    0    -1
 $EndComp
@@
 L Device:C_Small C1
 U 1 1 5BF4E13F
-P 2150 1800
-F 0 "C1" H 2200 1900 50  0000 L CNN
-F 1 "10u" H 2200 1750 50  0000 L CNN
-F 2 "Capacitor_SMD:C_0603_1608Metric_Pad1.05x0.95mm_HandSolder" H 2150 1800 50  0001 C CNN
-F 3 "~" H 2150 1800 50  0001 C CNN
-	1    2150 1800
+P 2150 1450
+F 0 "C1" H 2200 1550 50  0000 L CNN
+F 1 "10u" H 2200 1400 50  0000 L CNN
+F 2 "Capacitor_SMD:C_0603_1608Metric_Pad1.05x0.95mm_HandSolder" H 2150 1450 50  0001 C CNN
+F 3 "~" H 2150 1450 50  0001 C CNN
+	1    2150 1450
 	1    0    0    -1
 $EndComp
@@
 SW_Flag2
 Wire Notes Line
-	8190 4330 11225 4330
-Wire Notes Line
 	6970 6535 6970 7795
 Wire Notes Line
 	6970 7795 4095 7795
 Wire Notes Line
-	6970 6535 11220 6535
-Wire Notes Line
-	4095 470  4095 7795
-Wire Notes Line
-	470  3405 470  470
-Wire Notes Line
-	470  3405 8190 3405
-Wire Notes Line
-	470  470  11220 470
-Wire Notes Line
-	11220 470  11220 6535
-Wire Notes Line
-	4100 750  11220 750
-Wire Notes Line
-	4092 750  472  750
-Wire Notes Line
 	472  750  472  748
-Wire Notes Line
-	4098 3616 8192 3616
-Wire Notes Line
-	8190 6535 8190 470
-Wire Notes Line
-	8190 4500 11224 4500
-Wire Notes Line
-	11224 4500 11224 4494
 Connection ~ 8450 5900
 Wire Wire Line
@@
 L MRDT_Devices:OKI U2
 U 1 1 5C18C3BC
-P 2400 1750
-F 0 "U2" H 2450 1700 60  0001 C CNN
-F 1 "OKI" H 2600 2000 60  0000 C CNN
-F 2 "MRDT_Devices:OKI_Horizontal" H 2200 1650 60  0001 C CNN
-F 3 "" H 2200 1650 60  0001 C CNN
-	1    2400 1750
+P 2400 1400
+F 0 "U2" H 2450 1350 60  0001 C CNN
+F 1 "OKI" H 2600 1650 60  0000 C CNN
+F 2 "MRDT_Devices:OKI_Horizontal" H 2200 1300 60  0001 C CNN
+F 3 "" H 2200 1300 60  0001 C CNN
+	1    2400 1400
 	1    0    0    -1
 $EndComp
@@
 L MRDT_Devices:OKI U3
 U 1 1 5C18C438
-P 2400 2350
-F 0 "U3" H 2450 2300 60  0001 C CNN
-F 1 "OKI" H 2600 2600 60  0000 C CNN
-F 2 "MRDT_Devices:OKI_Horizontal" H 2200 2250 60  0001 C CNN
-F 3 "" H 2200 2250 60  0001 C CNN
-	1    2400 2350
+P 2400 2000
+F 0 "U3" H 2450 1950 60  0001 C CNN
+F 1 "OKI" H 2600 2250 60  0000 C CNN
+F 2 "MRDT_Devices:OKI_Horizontal" H 2200 1900 60  0001 C CNN
+F 3 "" H 2200 1900 60  0001 C CNN
+	1    2400 2000
 	1    0    0    -1
 $EndComp
@@
 L power:+5V #PWR0101
 U 1 1 5C28B373
-P 3000 1600
-F 0 "#PWR0101" H 3000 1450 50  0001 C CNN
-F 1 "+5V" H 2950 1750 50  0000 C CNN
-F 2 "" H 3000 1600 50  0001 C CNN
-F 3 "" H 3000 1600 50  0001 C CNN
-	1    3000 1600
-	1    0    0    -1
-$EndComp
-Wire Wire Line
-	3000 2550 3000 2500
+P 3000 1250
+F 0 "#PWR0101" H 3000 1100 50  0001 C CNN
+F 1 "+5V" H 2950 1400 50  0000 C CNN
+F 2 "" H 3000 1250 50  0001 C CNN
+F 3 "" H 3000 1250 50  0001 C CNN
+	1    3000 1250
+	1    0    0    -1
+$EndComp
+Wire Wire Line
+	3000 2200 3000 2150
 $Comp
 L power:+3.3V #PWR0105
 U 1 1 5C309CE1
-P 3000 2200
-F 0 "#PWR0105" H 3000 2050 50  0001 C CNN
-F 1 "+3.3V" H 2900 2350 50  0000 C CNN
-F 2 "" H 3000 2200 50  0001 C CNN
-F 3 "" H 3000 2200 50  0001 C CNN
-	1    3000 2200
-	1    0    0    -1
-$EndComp
-Connection ~ 3000 2250
-Connection ~ 2600 2550
-Wire Wire Line
-	3000 2250 3000 2300
-Wire Wire Line
-	3000 2200 3000 2250
-Wire Wire Line
-	2600 2550 3000 2550
-Wire Wire Line
-	3000 1600 3000 1650
-Connection ~ 3000 1650
-Connection ~ 2600 1950
-Wire Wire Line
-	2600 1950 3000 1950
-Wire Wire Line
-	3000 1700 3000 1650
+P 3000 1850
+F 0 "#PWR0105" H 3000 1700 50  0001 C CNN
+F 1 "+3.3V" H 2900 2000 50  0000 C CNN
+F 2 "" H 3000 1850 50  0001 C CNN
+F 3 "" H 3000 1850 50  0001 C CNN
+	1    3000 1850
+	1    0    0    -1
+$EndComp
+Connection ~ 3000 1900
+Connection ~ 2600 2200
 Wire Wire Line
 	3000 1900 3000 1950
+Wire Wire Line
+	3000 1850 3000 1900
+Wire Wire Line
+	2600 2200 3000 2200
+Wire Wire Line
+	3000 1250 3000 1300
+Connection ~ 3000 1300
+Connection ~ 2600 1600
+Wire Wire Line
+	2600 1600 3000 1600
+Wire Wire Line
+	3000 1350 3000 1300
+Wire Wire Line
+	3000 1550 3000 1600
 $Comp
 L Device:C_Small C2
 U 1 1 5BF4E0B2
-P 3000 1800
-F 0 "C2" H 3100 1850 50  0000 L CNN
-F 1 "10u" H 3100 1750 50  0000 L CNN
-F 2 "Capacitor_SMD:C_0603_1608Metric_Pad1.05x0.95mm_HandSolder" H 3000 1800 50  0001 C CNN
-F 3 "~" H 3000 1800 50  0001 C CNN
-	1    3000 1800
-	1    0    0    -1
-$EndComp
-Wire Wire Line
-	2200 2250 2150 2250
-Wire Wire Line
-	2150 2250 2150 2300
-Wire Wire Line
-	2150 2500 2150 2550
-Wire Wire Line
-	2600 2550 2150 2550
-Wire Wire Line
-	2150 1650 2150 1700
-Wire Wire Line
-	2150 1650 2200 1650
+P 3000 1450
+F 0 "C2" H 3100 1500 50  0000 L CNN
+F 1 "10u" H 3100 1400 50  0000 L CNN
+F 2 "Capacitor_SMD:C_0603_1608Metric_Pad1.05x0.95mm_HandSolder" H 3000 1450 50  0001 C CNN
+F 3 "~" H 3000 1450 50  0001 C CNN
+	1    3000 1450
+	1    0    0    -1
+$EndComp
+Wire Wire Line
+	2200 1900 2150 1900
 Wire Wire Line
 	2150 1900 2150 1950
 Wire Wire Line
-	2150 1950 2600 1950
-Wire Wire Line
-	2150 1650 2000 1650
-Connection ~ 2150 1650
-Connection ~ 2150 2250
-Wire Wire Line
-	3000 1950 3100 1950
-Connection ~ 3000 1950
-Connection ~ 3000 2550
-Wire Wire Line
-	2150 2550 1900 2550
-Connection ~ 2150 2550
+	2150 2150 2150 2200
+Wire Wire Line
+	2600 2200 2150 2200
+Wire Wire Line
+	2150 1300 2150 1350
+Wire Wire Line
+	2150 1300 2200 1300
+Wire Wire Line
+	2150 1550 2150 1600
+Wire Wire Line
+	2150 1600 2600 1600
+Wire Wire Line
+	2150 1300 2000 1300
+Connection ~ 2150 1300
+Connection ~ 2150 1900
+Wire Wire Line
+	3000 1600 3100 1600
+Connection ~ 3000 1600
+Connection ~ 3000 2200
+Wire Wire Line
+	2150 2200 1900 2200
+Connection ~ 2150 2200
 $Comp
 L power:GND #PWR0107
 U 1 1 5C5BBE3B
-P 3100 2550
-F 0 "#PWR0107" H 3100 2300 50  0001 C CNN
-F 1 "GND" H 3105 2377 50  0000 C CNN
-F 2 "" H 3100 2550 50  0001 C CNN
-F 3 "" H 3100 2550 50  0001 C CNN
-	1    3100 2550
-	1    0    0    -1
-$EndComp
-Wire Wire Line
-	3100 1950 3100 2550
-Connection ~ 3100 2550
-Wire Wire Line
-	3100 2550 3000 2550
-Wire Wire Line
-	2150 2250 2000 2250
+P 3100 2200
+F 0 "#PWR0107" H 3100 1950 50  0001 C CNN
+F 1 "GND" H 3105 2027 50  0000 C CNN
+F 2 "" H 3100 2200 50  0001 C CNN
+F 3 "" H 3100 2200 50  0001 C CNN
+	1    3100 2200
+	1    0    0    -1
+$EndComp
+Wire Wire Line
+	3100 1600 3100 2200
+Connection ~ 3100 2200
+Wire Wire Line
+	3100 2200 3000 2200
+Wire Wire Line
+	2150 1900 2000 1900
 $Comp
 L MRDT_Connectors:AndersonPP Conn1
 U 2 1 5BCC6C75
-P 1500 1750
-F 0 "Conn1" H 1600 2000 60  0000 C CNN
-F 1 "AndersonPP" H 950 1850 60  0001 C CNN
-F 2 "MRDT_Connectors:Anderson_2_Horisontal_Side_by_Side" H 1350 1200 60  0001 C CNN
-F 3 "" H 1350 1200 60  0001 C CNN
-	2    1500 1750
-	1    0    0    -1
-$EndComp
-Wire Wire Line
-	1900 1650 2000 1650
-Connection ~ 2000 1650
-Wire Wire Line
-	2000 1650 2000 2250
+P 1500 1400
+F 0 "Conn1" H 1600 1650 60  0000 C CNN
+F 1 "AndersonPP" H 950 1500 60  0001 C CNN
+F 2 "MRDT_Connectors:Anderson_2_Horisontal_Side_by_Side" H 1350 850 60  0001 C CNN
+F 3 "" H 1350 850 60  0001 C CNN
+	2    1500 1400
+	1    0    0    -1
+$EndComp
+Wire Wire Line
+	1900 1300 2000 1300
+Connection ~ 2000 1300
+Wire Wire Line
+	2000 1300 2000 1900
 Text Notes 6450 3900 0    50   ~ 0
 SPI 3
-Text Notes 6050 5750 0    50   ~ 0
-SPI 1
-Text Notes 4450 4400 0    50   ~ 0
-SPI 1\n
+Wire Notes Line
+	450  750  11250 750
+Wire Notes Line
+	8200 4300 11250 4300
+Wire Notes Line
+	8200 450  8200 6550
+Wire Notes Line
+	4150 450  4150 7800
+Wire Notes Line
+	4150 2800 450  2800
+Wire Notes Line
+	8200 4550 11250 4550
+Wire Notes Line
+	4150 3400 8200 3400
+Wire Notes Line
+	4150 3600 8200 3600
+Text Notes 7950 4400 2    50   ~ 0
+A14
+Text Notes 6500 4400 2    50   ~ 0
+A1
 $EndSCHEMATC

Commit message: finished PCB
Parts:
- removed Conn7, Conn8: Molex_SL_08, MRDT_Connectors:MOLEX_SL_08_Horizontal, symbol MRDT_Connectors:Molex_SL_08
- removed Conn9: Molex_SL_04, MRDT_Connectors:MOLEX_SL_04_Horizontal, symbol MRDT_Connectors:Molex_SL_04
- added D1: LED, Diode_SMD:D_0603_1608Metric_Pad1.05x0.95mm_HandSolder, symbol Device:LED
- added R14: 500, Resistor_SMD:R_0603_1608Metric_Pad1.05x0.95mm_HandSolder, symbol Device:R
- Conn5: value Molex_SL_05 -> Molex_SL_03; footprint MRDT_Connectors:MOLEX_SL_05_Horizontal -> MRDT_Connectors:MOLEX_SL_03_Horizontal; symbol MRDT_Connectors:Molex_SL_05 -> MRDT_Connectors:Molex_SL_03
Connections:
- net labels added: CCD_INT
- net labels removed: Bit0, Bit1, Bit10, Bit11, Bit12, Bit13, Bit14, Bit2, Bit3, Bit4, Bit5, Bit6, Bit7, Bit8, Bit9, CS, ICG, Master_CLOCK, SCLK, SDATA, Shift_Gate
- wire segments 152 -> 114
Other:
- note added: "CCD_TIVA"
- note added: "YELO"
- note removed: "CCD Breakout\n"
- note removed: "CCD Ouput Byte1"
- note removed: "CCD Output Byte2"
- note removed: "Charged Coupled Device"
- note removed: "SPI 3"
- moved on the sheet: D10, D11, D3, D4, D5, D6, D7, D8, D9, R1, R10, R11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

Commit message: updated CCD connector
Parts:
- Conn5: value Molex_SL_03 -> Molex_SL_04; footprint MRDT_Connectors:MOLEX_SL_03_Horizontal -> MRDT_Connectors:MOLEX_SL_04_Horizontal; symbol MRDT_Connectors:Molex_SL_03 -> MRDT_Connectors:Molex_SL_04
Connections:
- net labels added: CCD_OS
- wire segments 114 -> 106
Other:
- note added: "A10"
Changed lines of the file:
@@
 L power:+3.3V #PWR0116
 U 1 1 5BCFBAC2
-P 5050 1950
-F 0 "#PWR0116" H 5050 1800 50  0001 C CNN
-F 1 "+3.3V" H 5065 2123 50  0000 C CNN
-F 2 "" H 5050 1950 50  0001 C CNN
-F 3 "" H 5050 1950 50  0001 C CNN
-	1    5050 1950
+P 5050 1850
+F 0 "#PWR0116" H 5050 1700 50  0001 C CNN
+F 1 "+3.3V" H 5065 2023 50  0000 C CNN
+F 2 "" H 5050 1850 50  0001 C CNN
+F 3 "" H 5050 1850 50  0001 C CNN
+	1    5050 1850
 	1    0    0    -1
 $EndComp
@@
 AnalogOut
 $Comp
-L MRDT_Connectors:Molex_SL_03 Conn5
+L MRDT_Connectors:Molex_SL_04 Conn5
 U 1 1 5BF11252
 P 5300 2250
 F 0 "Conn5" H 5427 2558 60  0000 L CNN
-F 1 "Molex_SL_03" H 5427 2452 60  0000 L CNN
-F 2 "MRDT_Connectors:MOLEX_SL_03_Horizontal" H 5300 2250 60  0001 C CNN
+F 1 "Molex_SL_04" H 5427 2452 60  0000 L CNN
+F 2 "MRDT_Connectors:MOLEX_SL_04_Horizontal" H 5300 2250 60  0001 C CNN
 F 3 "" H 5300 2250 60  0001 C CNN
 	1    5300 2250
@@
 $EndComp
 Wire Wire Line
-	5050 2000 5100 2000
-Wire Wire Line
-	5050 2000 5050 1950
+	5050 1900 5100 1900
+Wire Wire Line
+	5050 1900 5050 1850
 Wire Wire Line
 	5050 2250 5050 2200
@@
 Wire Notes Line
 	472  750  472  748
-Connection ~ 8350 5900
-Wire Wire Line
-	8350 5900 8350 5950
-Connection ~ 8650 5900
-Wire Wire Line
-	8650 5900 8650 5950
-Connection ~ 8950 5900
-Wire Wire Line
-	8950 5900 8950 5950
-Connection ~ 9250 5900
-Wire Wire Line
-	9250 5900 9250 5950
-Connection ~ 9550 5900
-Wire Wire Line
-	9550 5900 9550 5950
-Connection ~ 9850 5900
-Wire Wire Line
-	9850 5900 9850 5950
-Connection ~ 10450 5900
-Wire Wire Line
-	10450 5900 10450 5950
-Connection ~ 10750 5900
-Wire Wire Line
-	10750 5900 10750 5950
-Connection ~ 11050 5900
-Wire Wire Line
-	11050 5900 11050 5950
 Text Notes 8140 7645 0    59   ~ 0
 12/19/18
@@
 Text Notes 10100 6300 0    50   ~ 0
 YELO
-Connection ~ 10150 5900
-Wire Wire Line
-	10150 5900 10150 5950
 Wire Wire Line
 	10150 5100 10150 5150
+Text GLabel 5050 2000 0    50   Output ~ 0
+CCD_OS
+Wire Wire Line
+	5100 2000 5050 2000
+Text GLabel 5850 6200 2    50   Input ~ 0
+CCD_OS
+Wire Wire Line
+	5800 6200 5850 6200
+Text Notes 6200 6250 0    50   ~ 0
+A10
 $EndSCHEMATC

Commit message: Modified CCD connector
Parts:
- Conn5: value Molex_SL_04 -> Molex_SL_05; footprint MRDT_Connectors:MOLEX_SL_04_Horizontal -> MRDT_Connectors:MOLEX_SL_05_Horizontal; symbol MRDT_Connectors:Molex_SL_04 -> MRDT_Connectors:Molex_SL_05
Connections:
- net CCD_INT: no longer Conn5.3, U1.PE0 (B1_3)
- net CCD_OS: now also Conn5.4; no longer Conn5.2
- net GND: now also Conn5.5; no longer Conn5.4
- net CCD_INT2: now reaches U1.PE1 (B1_4)
- net CCD_INT2: now also Conn5.2
- new net CCD_INT1: Conn5.3, U1.PE0 (B1_3)
Changed lines of the file:
@@
 Text GLabel 7700 5700 2    50   Output ~ 0
 UV_TOGGLE
-Text Notes 5250 1800 0    79   ~ 16
+Text Notes 5250 1700 0    79   ~ 16
 CCD_TIVA
 Text Notes 6600 1800 0    79   ~ 16
@@
 Wire Wire Line
 	5850 4350 5800 4350
-$Comp
-L power:+3.3V #PWR0116
-U 1 1 5BCFBAC2
-P 5050 1850
-F 0 "#PWR0116" H 5050 1700 50  0001 C CNN
-F 1 "+3.3V" H 5065 2023 50  0000 C CNN
-F 2 "" H 5050 1850 50  0001 C CNN
-F 3 "" H 5050 1850 50  0001 C CNN
-	1    5050 1850
-	1    0    0    -1
-$EndComp
 $Comp
 L power:GND #PWR0117
@@
 AnalogOut
 $Comp
-L MRDT_Connectors:Molex_SL_04 Conn5
+L MRDT_Connectors:Molex_SL_05 Conn5
 U 1 1 5BF11252
 P 5300 2250
 F 0 "Conn5" H 5427 2558 60  0000 L CNN
-F 1 "Molex_SL_04" H 5427 2452 60  0000 L CNN
-F 2 "MRDT_Connectors:MOLEX_SL_04_Horizontal" H 5300 2250 60  0001 C CNN
+F 1 "Molex_SL_05" H 5427 2452 60  0000 L CNN
+F 2 "MRDT_Connectors:MOLEX_SL_05_Horizontal" H 5300 2250 60  0001 C CNN
 F 3 "" H 5300 2250 60  0001 C CNN
 	1    5300 2250
 	1    0    0    -1
 $EndComp
-Wire Wire Line
-	5050 1900 5100 1900
-Wire Wire Line
-	5050 1900 5050 1850
 Wire Wire Line
 	5050 2250 5050 2200
@@
 Text Notes 6500 4400 2    50   ~ 0
 A1
-Text GLabel 5050 2100 0    50   Output ~ 0
-CCD_INT
+Text GLabel 5050 2000 0    50   Output ~ 0
+CCD_INT1
 Wire Wire Line
 	5100 2100 5050 2100
 Text GLabel 5850 4150 2    50   Input ~ 0
-CCD_INT
+CCD_INT1
 Wire Wire Line
 	5850 4150 5800 4150
@@
 Wire Wire Line
 	10150 5100 10150 5150
-Text GLabel 5050 2000 0    50   Output ~ 0
+Text GLabel 5050 2100 0    50   Output ~ 0
 CCD_OS
 Wire Wire Line
@@
 Text Notes 6200 6250 0    50   ~ 0
 A10
+Text GLabel 5050 1900 0    50   Output ~ 0
+CCD_INT2
+Wire Wire Line
+	5100 1900 5050 1900
+Text GLabel 5850 4250 2    50   Input ~ 0
+CCD_INT2
+Wire Wire Line
+	5800 4250 5850 4250
+$Comp
+L power:+3.3V #PWR?
+U 1 1 5C84A937
+P 5050 1750
+F 0 "#PWR?" H 5050 1600 50  0001 C CNN
+F 1 "+3.3V" H 5065 1923 50  0000 C CNN
+F 2 "" H 5050 1750 50  0001 C CNN
+F 3 "" H 5050 1750 50  0001 C CNN
+	1    5050 1750
+	1    0    0    -1
+$EndComp
+Wire Wire Line
+	5100 1800 5050 1800
+Wire Wire Line
+	5050 1800 5050 1750
 $EndSCHEMATC
