File: SRASensorBoard_Hardware/SRASensorBoard_Hardware.sch (KiCad schematic (older format))
At the start: 39 parts, among them U1 Tive Header, U2 OKI, U3 OKI

Commit message: fixed schematic
Parts:
- gave numbers to parts that had none: 2
Changed lines of the file:
@@
 YELO
 $Comp
-L power:GND #PWR?
+L power:GND #PWR0120
 U 1 1 5C8E01AB
 P 10450 5900
-F 0 "#PWR?" H 10450 5650 50  0001 C CNN
+F 0 "#PWR0120" H 10450 5650 50  0001 C CNN
 F 1 "GND" V 10455 5772 50  0000 R CNN
 F 2 "" H 10450 5900 50  0001 C CNN
@@
 	10450 5850 10450 5900
 $Comp
-L Device:LED D?
+L Device:LED D2
 U 1 1 5C8E01B2
 P 10450 5700
-F 0 "D?" H 10450 5800 50  0000 C CNN
+F 0 "D2" H 10450 5800 50  0000 C CNN
 F 1 "LED" H 10450 5600 50  0000 C CNN
 F 2 "Diode_SMD:D_0603_1608Metric_Pad1.05x0.95mm_HandSolder" H 10450 5700 50  0001 C CNN
@@
 	10450 5450 10450 5550
 $Comp
-L Device:R R?
+L Device:R R15
 U 1 1 5C8E01B9
 P 10450 5300
-F 0 "R?" V 10350 5300 50  0000 C CNN
+F 0 "R15" V 10350 5300 50  0000 C CNN
 F 1 "500" V 10450 5300 50  0000 C CNN
 F 2 "Resistor_SMD:R_0603_1608Metric_Pad1.05x0.95mm_HandSolder" V 10380 5300 50  0001 C CNN

Commit message: Rev 2 rework
Changed the connectors to vertical, retraced traces, etc.
Parts:
- Conn1: symbol MRDT_Connectors:AndersonPP -> SRASensorBoard_Hardware-rescue:AndersonPP-MRDT_Connectors
- Conn2, Conn4: footprint MRDT_Connectors:MOLEX_SL_04_Horizontal -> MRDT_Connectors:MOLEX_SL_04_Vertical; symbol MRDT_Connectors:Molex_SL_04 -> SRASensorBoard_Hardware-rescue:Molex_SL_04-MRDT_Connectors
- Conn3: footprint MRDT_Connectors:MOLEX_SL_03_Horizontal -> MRDT_Connectors:MOLEX_SL_03_Vertical; symbol MRDT_Connectors:Molex_SL_03 -> SRASensorBoard_Hardware-rescue:Molex_SL_03-MRDT_Connectors
- Conn5: footprint MRDT_Connectors:MOLEX_SL_05_Horizontal -> MRDT_Connectors:MOLEX_SL_05_Vertical; symbol MRDT_Connectors:Molex_SL_05 -> SRASensorBoard_Hardware-rescue:Molex_SL_05-MRDT_Connectors
- Conn6: footprint MRDT_Connectors:MOLEX_SL_02_Horizontal -> MRDT_Connectors:MOLEX_SL_02_Vertical; symbol MRDT_Connectors:Molex_SL_02 -> SRASensorBoard_Hardware-rescue:Molex_SL_02-MRDT_Connectors
- U1: symbol MRDT_Shields:TM4C129E_Launchpad -> SRASensorBoard_Hardware-rescue:TM4C129E_Launchpad-MRDT_Shields
- U2, U3: symbol MRDT_Devices:OKI -> SRASensorBoard_Hardware-rescue:OKI-MRDT_Devices
Other:
- moved on the sheet: D1, D10, D11, D2, D3, D4, D5, D6, D7, D8, D9, R1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
