File: SRASensorBoard_Hardware/SRA_Sensor_Board.kicad_pcb (KiCad board)
At the start: 2 copper layers, 70 parts, among them J1 USB_B_Micro, Q1 CSD17305Q5A, U1 LM3478MMX_NOPB, U2 OKI, U3 OKI, U4 TM4C129E_Launchpad, U5 MAX232, U6 IRF7821PbF

Commit message: Worked on some tracing
Commiting so I don't lose progress.
Parts:
- moved R22 162.0 mm to (68.6, 110.1), turned to 270 degrees
- moved R9 140.4 mm to (78.7, 110.1), turned to 270 degrees
- moved U5 135.8 mm to (85.1, 68.6)
- moved R10 129.9 mm to (83.8, 110.1), turned to 270 degrees
- moved R13 128.5 mm to (99.1, 110.1), turned to 270 degrees
- moved R11 115.7 mm to (88.9, 110.1), turned to 270 degrees
- moved R23 115.7 mm to (109.2, 110.1), turned to 270 degrees
- moved R7 115.5 mm to (104.1, 110.1), turned to 270 degrees
- moved R16 102.1 mm to (129.5, 110.1), turned to 270 degrees
- moved J1 96.3 mm to (184.2, 62.2), turned to 90 degrees
- moved C10 88.5 mm to (132.1, 80.9), turned to 270 degrees
- moved U2 87.1 mm to (100.3, 53.3), turned to 180 degrees
- moved R14 85.8 mm to (119.4, 110.1), turned to 270 degrees
- moved U3 85.7 mm to (113.0, 53.3), turned to 180 degrees
- moved R8 84.4 mm to (73.7, 110.1), turned to 270 degrees
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Routing:
- net GND: track 0.00 -> 120.7 mm, vias 0 -> 8
- net Net-(D1-Pad2): track 0.00 -> 23.0 mm
- net Net-(Q1-Pad4): track 0.00 -> 18.9 mm, vias 0 -> 2
- net Net-(C1-Pad1): track 0.00 -> 17.2 mm
- net +24V: track 0.00 -> 16.4 mm
- net Net-(Q1-Pad1): track 0.00 -> 13.3 mm
- net Net-(C3-Pad1): track 0.00 -> 10.1 mm
- net Net-(R1-Pad1): track 0.00 -> 8.68 mm
- net Net-(C8-Pad1): track 0.00 -> 6.60 mm
- net Net-(R5-Pad1): track 0.00 -> 4.43 mm
- net Net-(D9-Pad2): track 0.00 -> 2.85 mm
- net Net-(D8-Pad2): track 0.00 -> 2.85 mm
- net Net-(D7-Pad2): track 0.00 -> 2.85 mm
- net Net-(D6-Pad2): track 0.00 -> 2.85 mm
- net Net-(D5-Pad2): track 0.00 -> 2.85 mm
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- added copper zone on B.Cu, net GND
