File: SRASensorBoard_Hardware/_autosave-SRA_Sensor_Board.kicad_pcb (KiCad board)
At the start: 2 copper layers, 70 parts, among them J1 USB_B_Micro, Q1 CSD17305Q5A, U1 LM3478MMX_NOPB, U2 OKI, U3 OKI, U4 TM4C129E_Launchpad, U5 MAX232, U6 IRF7821PbF

Commit message: More Routing
mor
Parts:
- moved C12 86.4 mm to (104.1, 77.5), turned to 90 degrees
- moved Conn3 59.4 mm to (116.8, 68.6), turned to 180 degrees
- moved Conn1 58.5 mm to (116.8, 77.5), turned to 180 degrees
- moved Conn4 8.03 mm to (76.2, 80.0), turned to 180 degrees
Routing:
- net +5V: track 37.9 -> 250.7 mm
- net CCD_OS: track 0.00 -> 87.3 mm, vias 0 -> 2
- net +3V3: track 5.06 -> 72.3 mm, vias 0 -> 2
- net C02_In: track 0.00 -> 62.1 mm, vias 0 -> 2
- net +12V: track 50.0 -> 110.7 mm
- net C02_Out: track 0.00 -> 55.7 mm, vias 0 -> 2
- net GND: track 181.0 -> 217.9 mm, vias 12 -> 15
- net Flow_Output: track 0.00 -> 36.8 mm, vias 0 -> 2
- net Flow_Receive: track 0.00 -> 31.6 mm, vias 0 -> 2
- net CCD_INT1: track 0.00 -> 9.93 mm
- net CCD_INT2: track 0.00 -> 7.38 mm, vias 0 -> 2
- net Net-(D1-Pad2): track 23.0 -> 29.3 mm
- net LED_Enable: track 58.9 -> 55.6 mm
- net USB_Data_2: track 105.7 -> 106.8 mm
- net USB_Data_1: track 93.4 -> 94.3 mm, vias 0 -> 2
