File: SRASensorBoard_Hardware/_autosave-SRA_Sensor_Board.kicad_pcb (KiCad board)
At the start: 2 copper layers, 72 parts, among them J1 USB_A, Q1 BSS138, Q2 BSS138, Q3 BSS138, Q4 BSS138, U1 LT1910, U2 OKI, U3 OKI, U4 TM4C129E_Launchpad, U5 IRF7821PbF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

Commit message: Board Genral Layout
General layout is done. Components are organized into groups for easier design.
Parts:
- removed Conn7, Conn8: Boost GND, MRDT_Connectors:Anderson_2_Horizontal_Stacked
- Conn5: value 12v Boost -> BoostA
- Conn6: value 24v Boost -> BoostB
- moved Conn10 220.2 mm to (82.5, 77.5)
- moved Conn6 179.2 mm to (78.7, 72.4)
- moved Conn9 158.6 mm to (82.5, 86.4)
- moved Conn2 131.3 mm to (174.0, 41.9), turned to 180 degrees
- moved Conn5 108.8 mm to (174.0, 58.4), turned to 180 degrees
- moved U3 106.0 mm to (115.3, 58.4), turned to 180 degrees
- moved U2 104.3 mm to (126.2, 58.4), turned to 180 degrees
- moved J1 103.1 mm to (100.3, 52.1), turned to 180 degrees
- moved Conn11 77.1 mm to (151.1, 81.3), turned to 180 degrees
- moved U6 12.6 mm to (189.2, 137.2)
Connections:
- Conn5 pad 1: (no net) -> GND
- Conn6 pad 1: (no net) -> GND
