File: SRASensorBoard_Hardware/SRA_Sensor_Board.sch (KiCad schematic (older format))
At the start: 72 parts, among them J1 USB_A, Q1 BSS138, Q2 BSS138, Q3 BSS138, Q4 BSS138, U1 LT1910, U2 OKI, U3 OKI, U4 TM4C129E_Launchpad, U5 IRF7821PbF, U6 FT232RL

Commit message: Updates
Added footprints. Created new board. Something is up with the andersons.
Parts:
- U1: footprint (none) -> MRDT_ICs:SOIC127P599X175-8N
- U4: footprint MRDT_Shields:TM4C129E_Launchpad_FULL_THT_TOP -> MRDT_Shields:TM4C129E_Launchpad_FULL_THT_BOTTOM
- U5: footprint (none) -> MRDT_ICs:IRF7821PBF
Changed lines of the file:
@@
 F 0 "U4" H 11250 3550 60  0000 L CNN
 F 1 "TM4C129E_Launchpad" H 11000 3550 60  0001 L CNN
-F 2 "MRDT_Shields:TM4C129E_Launchpad_FULL_THT_TOP" H 11250 3600 60  0001 C CNN
+F 2 "MRDT_Shields:TM4C129E_Launchpad_FULL_THT_BOTTOM" H 11250 3600 60  0001 C CNN
 F 3 "" H 11250 3600 60  0001 C CNN
 	7    11250 3600
@@
 F 0 "U4" H 11850 3550 60  0000 C CNN
 F 1 "TM4C129E_Launchpad" H 12000 3550 60  0001 C CNN
-F 2 "MRDT_Shields:TM4C129E_Launchpad_FULL_THT_TOP" H 11750 3600 60  0001 C CNN
+F 2 "MRDT_Shields:TM4C129E_Launchpad_FULL_THT_BOTTOM" H 11750 3600 60  0001 C CNN
 F 3 "" H 11750 3600 60  0001 C CNN
 	8    11750 3600
@@
 F 0 "U4" H 11850 2050 60  0000 C CNN
 F 1 "TM4C129E_Launchpad" H 12000 2050 60  0001 C CNN
-F 2 "MRDT_Shields:TM4C129E_Launchpad_FULL_THT_TOP" H 11750 2100 60  0001 C CNN
+F 2 "MRDT_Shields:TM4C129E_Launchpad_FULL_THT_BOTTOM" H 11750 2100 60  0001 C CNN
 F 3 "" H 11750 2100 60  0001 C CNN
 	4    11750 2100
@@
 F 0 "U4" H 11250 2050 60  0000 L CNN
 F 1 "TM4C129E_Launchpad" H 11000 2050 60  0001 L CNN
-F 2 "MRDT_Shields:TM4C129E_Launchpad_FULL_THT_TOP" H 11250 2100 60  0001 C CNN
+F 2 "MRDT_Shields:TM4C129E_Launchpad_FULL_THT_BOTTOM" H 11250 2100 60  0001 C CNN
 F 3 "" H 11250 2100 60  0001 C CNN
 	3    11250 2100
@@
 F 0 "U4" H 10050 2050 60  0000 C CNN
 F 1 "TM4C129E_Launchpad" H 10200 2050 60  0001 C CNN
-F 2 "MRDT_Shields:TM4C129E_Launchpad_FULL_THT_TOP" H 9950 2100 60  0001 C CNN
+F 2 "MRDT_Shields:TM4C129E_Launchpad_FULL_THT_BOTTOM" H 9950 2100 60  0001 C CNN
 F 3 "" H 9950 2100 60  0001 C CNN
 	2    9950 2100
@@
 F 0 "U4" H 9450 2050 60  0000 L CNN
 F 1 "TM4C129E_Launchpad" H 9200 2050 60  0001 L CNN
-F 2 "MRDT_Shields:TM4C129E_Launchpad_FULL_THT_TOP" H 9450 2100 60  0001 C CNN
+F 2 "MRDT_Shields:TM4C129E_Launchpad_FULL_THT_BOTTOM" H 9450 2100 60  0001 C CNN
 F 3 "" H 9450 2100 60  0001 C CNN
 	1    9450 2100
@@
 F 0 "U4" H 9450 3550 60  0000 L CNN
 F 1 "TM4C129E_Launchpad" H 9250 3550 60  0001 L CNN
-F 2 "MRDT_Shields:TM4C129E_Launchpad_FULL_THT_TOP" H 9450 3600 60  0001 C CNN
+F 2 "MRDT_Shields:TM4C129E_Launchpad_FULL_THT_BOTTOM" H 9450 3600 60  0001 C CNN
 F 3 "" H 9450 3600 60  0001 C CNN
 	5    9450 3600
@@
 F 0 "U4" H 10050 3550 60  0000 C CNN
 F 1 "TM4C129E_Launchpad" H 10150 3550 60  0001 C CNN
-F 2 "MRDT_Shields:TM4C129E_Launchpad_FULL_THT_TOP" H 9950 3600 60  0001 C CNN
+F 2 "MRDT_Shields:TM4C129E_Launchpad_FULL_THT_BOTTOM" H 9950 3600 60  0001 C CNN
 F 3 "" H 9950 3600 60  0001 C CNN
 	6    9950 3600
@@
 F 0 "U5" H 4100 7613 60  0000 C CNN
 F 1 "IRF7821PbF" H 4100 7719 60  0000 C CNN
-F 2 "" H 3750 7800 60  0001 C CNN
+F 2 "MRDT_ICs:IRF7821PBF" H 3750 7800 60  0001 C CNN
 F 3 "" H 3750 7800 60  0001 C CNN
 	1    3750 7800
@@
 F 0 "U1" H 2075 8937 60  0000 C CNN
 F 1 "LT1910" H 2075 8831 60  0000 C CNN
-F 2 "" H 1700 8250 60  0001 C CNN
+F 2 "MRDT_ICs:SOIC127P599X175-8N" H 1700 8250 60  0001 C CNN
 F 3 "" H 1700 8250 60  0001 C CNN
 	1    1700 8250
