File: SRASensorBoard_Hardware/SRA_Sensor_Board.sch (KiCad schematic (older format))
At the start: 28 parts

Commit message: Revert "new sensor rev 2"
This reverts commit 156ab373f26da52bc01a01f00cdb696ec9d5eefa.
Parts:
- added C1, C2: 47pF, Capacitor_SMD:C_0603_1608Metric_Pad1.05x0.95mm_HandSolder, symbol Device:C
- added C3: 100nf, Capacitor_SMD:C_0603_1608Metric_Pad1.05x0.95mm_HandSolder, symbol Device:C
- added C4, C5, C6, C7: 10uF, Capacitor_SMD:C_0603_1608Metric_Pad1.05x0.95mm_HandSolder, symbol Device:C
- added Conn1, Conn3: Molex_SL_04, MRDT_Connectors:MOLEX_SL_04_Vertical, symbol MRDT_Connectors:Molex_SL_04
- added Conn2: AndersonPP, MRDT_Connectors:Anderson_2_Horizontal_Side_by_Side, symbol MRDT_Connectors:AndersonPP
- added Conn5: Boost 12V, MRDT_Connectors:Anderson_2_Horizontal_Side_by_Side, symbol MRDT_Connectors:AndersonPP
- added Conn6: Boost 24V, MRDT_Connectors:Anderson_2_Horizontal_Side_by_Side, symbol MRDT_Connectors:AndersonPP
- added Conn7: UV_led, MRDT_Connectors:Anderson_2_Horizontal_Side_by_Side, symbol MRDT_Connectors:AndersonPP
- added J1: USB_A, custom:292303-1, symbol Connector:USB_A
- added Q1, Q2, Q3, Q4: BSS138, Package_TO_SOT_SMD:SOT-23, symbol Transistor_FET:BSS138
- added Q5: Q_PMOS_GDS, Package_TO_SOT_SMD:TO-252-2, symbol Device:Q_PMOS_GDS
- added Q6: Q_NMOS_GSD, Package_TO_SOT_SMD:SOT-23, symbol Device:Q_NMOS_GSD
- added R1, R2, R21, R25, R26, R27, R5, R6: 10K, Resistor_SMD:R_0603_1608Metric_Pad1.05x0.95mm_HandSolder, symbol Device:R
- added R28, R29: 22k, Resistor_SMD:R_0603_1608Metric_Pad1.05x0.95mm_HandSolder, symbol Device:R
- added R3: 4, Resistor_THT:R_Axial_DIN0414_L11.9mm_D4.5mm_P15.24mm_Horizontal, symbol Device:R
- added R30, R34: 10k, Resistor_SMD:R_0603_1608Metric_Pad1.05x0.95mm_HandSolder, symbol Device:R
- added R31, R32: 27, Resistor_SMD:R_0603_1608Metric_Pad1.05x0.95mm_HandSolder, symbol Device:R
- added R33: 4.7k, Resistor_SMD:R_0603_1608Metric_Pad1.05x0.95mm_HandSolder, symbol Device:R
- added U1: FT230XS, Package_SO:SSOP-16_3.9x4.9mm_P0.635mm, symbol Interface_USB:FT230XS
- added U2, U3: OKI, MRDT_Devices:OKI_Horizontal, symbol MRDT_Devices:OKI
- added U4: TM4C129E_Launchpad, MRDT_Shields:TM4C129E_Launchpad_FULL_THT_BOTTOM, symbol SRA_Sensor_Board-rescue:TM4C129E_Launchpad-MRDT_Shields-SRA_Sensor_Board-rescue
Connections:
- net +12V: now also C4.1, C5.1, Conn2.2 (V+Log), Conn5.2 (V+Log), U2.1 (Vi), U3.1 (Vi)
- net +24V: now also Conn6.2 (V+Log), Q5.3 (S), R28.1
- net +3V3: now also C7.1, Q1.1 (G), Q2.1 (G), Q3.1 (G), Q4.1 (G), R1.1, R2.1, R21.1, R25.1, U1.12 (VCC), U3.3 (Vo), U4.+3V3 (A1_1), U4.+3V3 (A2_1)
- net +5V: now also C6.1, Conn1.1, Conn3.1, J1.1 (VBUS), R26.1, R27.1, R33.2, R5.1, R6.1, U2.3 (Vo), U4.+5V (B1_1), U4.+5V (B2_1)
- net C02_RX: now also Conn3.4, Q2.3 (D), R6.2
- net C02_TX: now also Conn3.3, Q4.3 (D), R27.2
- net GND: now also C1.2, C2.2, C3.2, C4.2, C5.2, C6.2, C7.2, Conn1.2, Conn2.1 (GND), Conn3.2, Conn5.1 (GND), Conn6.1 (GND), Conn7.1 (GND), J1.4 (GND), Q6.2 (S), R30.1, R34.2, U1.13 (GND), U1.5 (GND), U2.2 (GND), U3.2 (GND), U4.GND (B1_2), U4.GND (B2_2), U4.GND (D1_1), U4.GND (D2_1)
- net LED_Enable: now also Q6.1 (G), R30.2, U4.PP5 (D2_3)
- net O2_RX: now also Conn1.4, Q1.3 (D), R5.2
- net O2_TX: now also Conn1.3, Q3.3 (D), R26.2
- net SW_ERROR: now also U4.PN4 (A2_10)
- net SW_Flag1: now also U4.PP4 (A2_8)
- net SW_Flag2: now also U4.PN5 (A2_9)
- net TIVA_USB_RX: now also U1.1 (TXD), U4.PC6 (A1_5)
- net TIVA_USB_TX: now also U1.4 (RXD), U4.PC7 (A1_8)
- new net: Conn7.2 (V+Log), R3.2
- new net: Q6.3 (D), R29.2
- new net: Q5.1 (G), R28.2, R29.1
- new net: Q5.2 (D), R3.1
- new net: C3.1, U1.10 (3V3OUT), U1.11 (~RESET), U1.3 (VCCIO)
- new net: R33.1, R34.1, U1.16 (CBUS3)
- new net: R32.1, U1.8 (USBDP)
- new net: R31.1, U1.9 (USBDM)
- new net Reset: U4.PM3 (D1_2)
- new net TIVA_CO2_RX: Q4.2 (S), R25.2, U4.PC4 (A1_3)
- new net TIVA_CO2_TX: Q2.2 (S), R2.2, U4.PC5 (A1_4)
- new net TIVA_O2_RX: Q3.2 (S), R21.2, U4.PK0 (B2_5)
- new net TIVA_O2_TX: Q1.2 (S), R1.2, U4.PK1 (B2_6)
- new net USB_Data+: C2.1, J1.3 (D+), R32.2
- new net USB_Data-: C1.1, J1.2 (D-), R31.2
- no-connect marks 0 -> 61
Other:
- note added: "CO2_Sensor\n"
- note added: "INPUT"
- note added: "Methane Sensor"
- note added: "Methane Sensor USB A\n"
- note added: "NGM_1"
- note added: "O2 Sensor"
- note added: "OUTPUT"
- note added: "Off Board Boost Converter"
- note added: "Power\n"
- note added: "Sensors\n"
- note added: "Serial 4"
- note added: "Serial 5"
- note added: "Serial 7"
- note added: "TIVA"
- note added: "UV_LED"
- note removed: "SICENCE SENSOR BOARD REV2"
- moved on the sheet: D10, D11, D15, D16, D17, D18, D2, D3, D4, D5, D6, D7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
