File: SRASensorBoard_Hardware/_autosave-SRA_Sensor_Board.sch (KiCad schematic (older format))
At the start: 72 parts, among them J1 USB_A, Q1 BSS138, Q2 BSS138, Q3 BSS138, Q4 BSS138, U1 LT1910, U2 OKI, U3 OKI, U4 TM4C129E_Launchpad, U5 IRF7821PbF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

Commit message: Board Genral Layout
General layout is done. Components are organized into groups for easier design.
Parts:
- Conn5: value 12v Boost -> BoostA
- Conn5: renamed from Conn7; value 12v Boost GND -> BoostA
- Conn6: value 24v Boost -> BoostB
- Conn6: renamed from Conn8; value 24v Boost GND -> BoostB
Changed lines of the file:
@@
 P 1650 6400
 F 0 "Conn5" H 1858 6787 60  0000 C CNN
-F 1 "12v Boost" H 1858 6681 60  0000 C CNN
+F 1 "BoostA" H 1858 6681 60  0000 C CNN
 F 2 "MRDT_Connectors:Anderson_2_Horizontal_Side_by_Side" H 1500 5850 60  0001 C CNN
 F 3 "" H 1500 5850 60  0001 C CNN
@@
 P 1650 6850
 F 0 "Conn6" H 1858 7237 60  0000 C CNN
-F 1 "24v Boost" H 1858 7131 60  0000 C CNN
+F 1 "BoostB" H 1858 7131 60  0000 C CNN
 F 2 "MRDT_Connectors:Anderson_2_Horizontal_Side_by_Side" H 1500 6300 60  0001 C CNN
 F 3 "" H 1500 6300 60  0001 C CNN
@@
 $EndComp
 $Comp
-L MRDT_Connectors:AndersonPP Conn7
+L MRDT_Connectors:AndersonPP Conn5
 U 1 1 5E1070D1
 P 2500 6400
-F 0 "Conn7" H 2708 6787 60  0000 C CNN
-F 1 "12v Boost GND" H 2708 6681 60  0000 C CNN
+F 0 "Conn5" H 2708 6787 60  0000 C CNN
+F 1 "BoostA" H 2708 6681 60  0000 C CNN
 F 2 "MRDT_Connectors:Anderson_2_Horizontal_Side_by_Side" H 2350 5850 60  0001 C CNN
 F 3 "" H 2350 5850 60  0001 C CNN
@@
 	3050 6300 2900 6300
 $Comp
-L MRDT_Connectors:AndersonPP Conn8
+L MRDT_Connectors:AndersonPP Conn6
 U 1 1 5E112038
 P 2500 6850
-F 0 "Conn8" H 2708 7237 60  0000 C CNN
-F 1 "24v Boost GND" H 2708 7131 60  0000 C CNN
+F 0 "Conn6" H 2708 7237 60  0000 C CNN
+F 1 "BoostB" H 2708 7131 60  0000 C CNN
 F 2 "MRDT_Connectors:Anderson_2_Horizontal_Side_by_Side" H 2350 6300 60  0001 C CNN
 F 3 "" H 2350 6300 60  0001 C CNN
