File: Hardware/SRASensorBoard_Hardware/SENSORS.sch (KiCad schematic (older format))
At the start: 75 parts, among them J1 USB_A, Q1 BSS138, Q10 BSS138, Q11 BSS138, Q12 BSS138, Q13 BSS138, Q2 BSS138, Q3 BSS138, Q4 BSS138, Q5 BSS138, Q6 BSS138, Q9 BSS138, U3 FT230XS

Commit message: Fixed some library issues
Parts:
- C5, C6, C7, C9: footprint Capacitor_SMD:C_0603_1608Metric_Pad1.05x0.95mm_HandSolder -> Capacitor_SMD:C_0603_1608Metric_Pad1.08x0.95mm_HandSolder
- C8: symbol Device:CP1_Small -> Device:C_Polarized_Small_US
- FB1: footprint Resistor_SMD:R_0805_2012Metric_Pad1.15x1.40mm_HandSolder -> Resistor_SMD:R_0805_2012Metric_Pad1.20x1.40mm_HandSolder; symbol Device:Ferrite_Bead_Small -> Device:FerriteBead_Small
- R1, R13, R14, R15, R16, R17, R18, R19, R2, R20, R21, R22, R23, R24, R25, R26, R27, R28, R29, R30, R41, R42, R43, R44, R45, R46, R47, R48, R7, R8: footprint Resistor_SMD:R_0603_1608Metric_Pad1.05x0.95mm_HandSolder -> Resistor_SMD:R_0603_1608Metric_Pad0.98x0.95mm_HandSolder
- R10, R31, R32, R5, R6, R9: value 330 -> 480; footprint Resistor_SMD:R_0603_1608Metric_Pad1.05x0.95mm_HandSolder -> Resistor_SMD:R_0603_1608Metric_Pad0.98x0.95mm_HandSolder
- R11, R12: value 330 -> 1K; footprint Resistor_SMD:R_0603_1608Metric_Pad1.05x0.95mm_HandSolder -> Resistor_SMD:R_0603_1608Metric_Pad0.98x0.95mm_HandSolder
Connections:
- net GND: now also J1.5 (Shield)
- no-connect marks 7 -> 6
