File: Hardware/SRASensorBoard_Hardware/SENSORS.sch (KiCad schematic (older format))
At the start: 75 parts, among them J1 USB_A, Q1 BSS138, Q10 BSS138, Q11 BSS138, Q12 BSS138, Q13 BSS138, Q2 BSS138, Q3 BSS138, Q4 BSS138, Q5 BSS138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

Commit message: Finished BOM
Parts:
- D10, D11, D12, D13, D14, D15, D16, D17, D18, D7, D8, D9: value LED -> Blue
Changed lines of the file:
@@
 AR Path="/5F841BF9/5FAD79F1" Ref="D7"  Part="1"
 F 0 "D7" V 2439 1233 50  0000 R CNN
-F 1 "LED" V 2348 1233 50  0000 R CNN
+F 1 "Blue" V 2348 1233 50  0000 R CNN
 F 2 "Diode_SMD:D_0603_1608Metric_Pad1.05x0.95mm_HandSolder" H 2400 1350 50  0001 C CNN
 F 3 "~" H 2400 1350 50  0001 C CNN
@@
 AR Path="/5F841BF9/5FAD7A05" Ref="D8"  Part="1"
 F 0 "D8" V 2439 1558 50  0000 R CNN
-F 1 "LED" V 2348 1558 50  0000 R CNN
+F 1 "Blue" V 2348 1558 50  0000 R CNN
 F 2 "Diode_SMD:D_0603_1608Metric_Pad1.05x0.95mm_HandSolder" H 2400 1675 50  0001 C CNN
 F 3 "~" H 2400 1675 50  0001 C CNN
@@
 AR Path="/5F841BF9/5FC31493" Ref="D11"  Part="1"
 F 0 "D11" V 2464 2558 50  0000 R CNN
-F 1 "LED" V 2373 2558 50  0000 R CNN
+F 1 "Blue" V 2373 2558 50  0000 R CNN
 F 2 "Diode_SMD:D_0603_1608Metric_Pad1.05x0.95mm_HandSolder" H 2425 2675 50  0001 C CNN
 F 3 "~" H 2425 2675 50  0001 C CNN
@@
 AR Path="/5F841BF9/5FC314A7" Ref="D12"  Part="1"
 F 0 "D12" V 2464 2883 50  0000 R CNN
-F 1 "LED" V 2373 2883 50  0000 R CNN
+F 1 "Blue" V 2373 2883 50  0000 R CNN
 F 2 "Diode_SMD:D_0603_1608Metric_Pad1.05x0.95mm_HandSolder" H 2425 3000 50  0001 C CNN
 F 3 "~" H 2425 3000 50  0001 C CNN
@@
 AR Path="/5F841BF9/5FC8B337" Ref="D9"  Part="1"
 F 0 "D9" V 2439 3883 50  0000 R CNN
-F 1 "LED" V 2348 3883 50  0000 R CNN
+F 1 "Blue" V 2348 3883 50  0000 R CNN
 F 2 "Diode_SMD:D_0603_1608Metric_Pad1.05x0.95mm_HandSolder" H 2400 4000 50  0001 C CNN
 F 3 "~" H 2400 4000 50  0001 C CNN
@@
 AR Path="/5F841BF9/5FC8B34B" Ref="D10"  Part="1"
 F 0 "D10" V 2439 4208 50  0000 R CNN
-F 1 "LED" V 2348 4208 50  0000 R CNN
+F 1 "Blue" V 2348 4208 50  0000 R CNN
 F 2 "Diode_SMD:D_0603_1608Metric_Pad1.05x0.95mm_HandSolder" H 2400 4325 50  0001 C CNN
 F 3 "~" H 2400 4325 50  0001 C CNN
@@
 AR Path="/5F841BF9/5FCC13BC" Ref="D13"  Part="1"
 F 0 "D13" V 2464 5233 50  0000 R CNN
-F 1 "LED" V 2373 5233 50  0000 R CNN
+F 1 "Blue" V 2373 5233 50  0000 R CNN
 F 2 "Diode_SMD:D_0603_1608Metric_Pad1.05x0.95mm_HandSolder" H 2425 5350 50  0001 C CNN
 F 3 "~" H 2425 5350 50  0001 C CNN
@@
 AR Path="/5F841BF9/5FCC13D0" Ref="D14"  Part="1"
 F 0 "D14" V 2464 5558 50  0000 R CNN
-F 1 "LED" V 2373 5558 50  0000 R CNN
+F 1 "Blue" V 2373 5558 50  0000 R CNN
 F 2 "Diode_SMD:D_0603_1608Metric_Pad1.05x0.95mm_HandSolder" H 2425 5675 50  0001 C CNN
 F 3 "~" H 2425 5675 50  0001 C CNN
@@
 AR Path="/5F841BF9/5FD3ACB3" Ref="D15"  Part="1"
 F 0 "D15" V 2464 6633 50  0000 R CNN
-F 1 "LED" V 2373 6633 50  0000 R CNN
+F 1 "Blue" V 2373 6633 50  0000 R CNN
 F 2 "Diode_SMD:D_0603_1608Metric_Pad1.05x0.95mm_HandSolder" H 2425 6750 50  0001 C CNN
 F 3 "~" H 2425 6750 50  0001 C CNN
@@
 AR Path="/5F841BF9/5FD3ACC7" Ref="D16"  Part="1"
 F 0 "D16" V 2464 6958 50  0000 R CNN
-F 1 "LED" V 2373 6958 50  0000 R CNN
+F 1 "Blue" V 2373 6958 50  0000 R CNN
 F 2 "Diode_SMD:D_0603_1608Metric_Pad1.05x0.95mm_HandSolder" H 2425 7075 50  0001 C CNN
 F 3 "~" H 2425 7075 50  0001 C CNN
@@
 AR Path="/5F841BF9/5FDDCD41" Ref="D17"  Part="1"
 F 0 "D17" V 8789 1183 50  0000 R CNN
-F 1 "LED" V 8698 1183 50  0000 R CNN
+F 1 "Blue" V 8698 1183 50  0000 R CNN
 F 2 "Diode_SMD:D_0603_1608Metric_Pad1.05x0.95mm_HandSolder" H 8750 1300 50  0001 C CNN
 F 3 "~" H 8750 1300 50  0001 C CNN
@@
 AR Path="/5F841BF9/5FDDCD33" Ref="D18"  Part="1"
 F 0 "D18" V 8789 1533 50  0000 R CNN
-F 1 "LED" V 8698 1533 50  0000 R CNN
+F 1 "Blue" V 8698 1533 50  0000 R CNN
 F 2 "Diode_SMD:D_0603_1608Metric_Pad1.05x0.95mm_HandSolder" H 8750 1650 50  0001 C CNN
 F 3 "~" H 8750 1650 50  0001 C CNN
