File: Hardware/SRASensorBoard_Hardware/TIVA.sch (KiCad schematic (older format))
At the start: 8 parts

Commit message: Sciency stuff for the board
finished!
Parts:
- added D? (x3): LED, Diode_SMD:D_0603_1608Metric_Pad1.05x0.95mm_HandSolder, symbol Device:LED
- added R? (x3): 330, Resistor_SMD:R_0603_1608Metric_Pad1.05x0.95mm_HandSolder, symbol Device:R
Connections:
- net GND: now also D?.1 (K), D?.1 (K), D?.1 (K)
- net SW_ERROR: now also R?.1
- net SW_Flag1: now also R?.1
- net SW_Flag2: now also R?.1
- net NO_SCL: now reaches U?.PB2 (A1_9)
- net NO_SDA: now reaches U?.PB3 (A1_10)
- net N2O_RX: now reaches U?.PP0 (A2_3)
- net N2O_TX: now reaches U?.PP1 (A2_4)
- net NO2_RX: now reaches U?.PA4 (B2_9)
- net NO2_TX: now reaches U?.PA5 (B2_10)
- new net: D?.2 (A), R?.2 (x3)
- no-connect marks 61 -> 55
Other:
- note added: "BLU"
- note added: "RED\n"
- note added: "SDA/SCL 0\n\n"
- note added: "Serial 3\n"
- note added: "Serial 6\n"
Changed lines of the file:
@@
 Text GLabel 7150 4100 2    50   Output ~ 0
 LED_Enable
-Text GLabel 4300 4800 0    50   Output ~ 0
+Text GLabel 4225 5275 0    50   Output ~ 0
 SW_ERROR
-Text GLabel 4300 4700 0    50   Output ~ 0
+Text GLabel 4200 4900 0    50   Output ~ 0
 SW_Flag2
-Text GLabel 4300 4600 0    50   Output ~ 0
+Text GLabel 4200 4500 0    50   Output ~ 0
 SW_Flag1
 Wire Wire Line
@@
 NoConn ~ 5300 4200
 NoConn ~ 5300 4500
-NoConn ~ 5300 4700
-NoConn ~ 5300 4800
 NoConn ~ 6200 4800
 NoConn ~ 6200 4700
@@
 NoConn ~ 6200 3200
 NoConn ~ 6200 3300
-NoConn ~ 4400 3300
-NoConn ~ 4400 3200
 NoConn ~ 4400 3000
 NoConn ~ 4400 2500
@@
 	4300 4600 4400 4600
 Wire Wire Line
-	4300 4700 4400 4700
-Wire Wire Line
 	4300 4800 4400 4800
 NoConn ~ 4400 4400
 NoConn ~ 4400 4300
-NoConn ~ 4400 4000
 Wire Wire Line
 	4300 3900 4400 3900
@@
 Wire Wire Line
 	5300 2500 5950 2500
-NoConn ~ 4400 4200
-NoConn ~ 4400 4100
 Text GLabel 7150 2500 2    50   Output ~ 0
 Reset
@@
 NoConn ~ 5300 2700
 NoConn ~ 5300 4600
+Text GLabel 4175 3325 0    50   Input ~ 0
+NO_SCL
+Text Notes 3775 3325 0    50   ~ 0
+SDA/SCL 0\n\n
+Text GLabel 4175 3425 0    50   Input ~ 0
+NO_SDA
+NoConn ~ 4400 4000
+Wire Wire Line
+	4400 4100 4150 4100
+Text GLabel 4150 4100 0    50   Input ~ 0
+N2O_RX
+Wire Wire Line
+	4400 4200 4150 4200
+Text GLabel 4150 4200 0    50   Output ~ 0
+N2O_TX
+Text Notes 3825 4000 0    50   ~ 0
+Serial 6\n
+Wire Wire Line
+	4400 3200 4250 3200
+Wire Wire Line
+	4250 3200 4250 3325
+Wire Wire Line
+	4250 3325 4175 3325
+Wire Wire Line
+	4400 3300 4300 3300
+Wire Wire Line
+	4300 3300 4300 3425
+Wire Wire Line
+	4300 3425 4175 3425
+Text GLabel 5475 4700 2    50   Input ~ 0
+NO2_RX
+Text GLabel 5475 4800 2    50   Output ~ 0
+NO2_TX
+Wire Wire Line
+	5300 4700 5475 4700
+Wire Wire Line
+	5300 4800 5475 4800
+Text Notes 5500 4625 0    50   ~ 0
+Serial 3\n
+$Comp
+L Device:LED D?
+U 1 1 605279AE
+P 3300 5050
+AR Path="/605279AE" Ref="D?"  Part="1"
+AR Path="/5F841BF9/605279AE" Ref="D?"  Part="1"
+AR Path="/5F8FEC08/605279AE" Ref="D?"  Part="1"
+F 0 "D?" V 3339 4933 50  0000 R CNN
+F 1 "LED" V 3248 4933 50  0000 R CNN
+F 2 "Diode_SMD:D_0603_1608Metric_Pad1.05x0.95mm_HandSolder" H 3300 5050 50  0001 C CNN
+F 3 "~" H 3300 5050 50  0001 C CNN
+	1    3300 5050
+	1    0    0    -1
+$EndComp
+$Comp
+L Device:R R?
+U 1 1 605279B4
+P 3700 5050
+AR Path="/605279B4" Ref="R?"  Part="1"
+AR Path="/5F841BF9/605279B4" Ref="R?"  Part="1"
+AR Path="/5F8FEC08/605279B4" Ref="R?"  Part="1"
+F 0 "R?" H 3770 5096 50  0000 L CNN
+F 1 "330" H 3770 5005 50  0000 L CNN
+F 2 "Resistor_SMD:R_0603_1608Metric_Pad1.05x0.95mm_HandSolder" V 3630 5050 50  0001 C CNN
+F 3 "~" H 3700 5050 50  0001 C CNN
+	1    3700 5050
+	0    1    1    0
+$EndComp
+Text Notes 2900 5000 3    50   ~ 0
+RED\n
+Wire Wire Line
+	3450 5050 3550 5050
+$Comp
+L Device:LED D?
+U 1 1 605279BE
+P 3300 4350
+AR Path="/605279BE" Ref="D?"  Part="1"
+AR Path="/5F841BF9/605279BE" Ref="D?"  Part="1"
+AR Path="/5F8FEC08/605279BE" Ref="D?"  Part="1"
+F 0 "D?" V 3339 4233 50  0000 R CNN
+F 1 "LED" V 3248 4233 50  0000 R CNN
+F 2 "Diode_SMD:D_0603_1608Metric_Pad1.05x0.95mm_HandSolder" H 3300 4350 50  0001 C CNN
+F 3 "~" H 3300 4350 50  0001 C CNN
+	1    3300 4350
+	1    0    0    -1
+$EndComp
+$Comp
+L Device:R R?
+U 1 1 605279C4
+P 3700 4350
+AR Path="/605279C4" Ref="R?"  Part="1"
+AR Path="/5F841BF9/605279C4" Ref="R?"  Part="1"
+AR Path="/5F8FEC08/605279C4" Ref="R?"  Part="1"
+F 0 "R?" H 3770 4396 50  0000 L CNN
+F 1 "330" H 3770 4305 50  0000 L CNN
+F 2 "Resistor_SMD:R_0603_1608Metric_Pad1.05x0.95mm_HandSolder" V 3630 4350 50  0001 C CNN
+F 3 "~" H 3700 4350 50  0001 C CNN
+	1    3700 4350
+	0    1    1    0
+$EndComp
+Text Notes 2900 4300 3    50   ~ 0
+BLU
+Wire Wire Line
+	3450 4350 3550 4350
+$Comp
+L Device:LED D?
+U 1 1 605279CE
+P 3300 4700
+AR Path="/605279CE" Ref="D?"  Part="1"
+AR Path="/5F841BF9/605279CE" Ref="D?"  Part="1"
+AR Path="/5F8FEC08/605279CE" Ref="D?"  Part="1"
+F 0 "D?" V 3339 4583 50  0000 R CNN
+F 1 "LED" V 3248 4583 50  0000 R CNN
+F 2 "Diode_SMD:D_0603_1608Metric_Pad1.05x0.95mm_HandSolder" H 3300 4700 50  0001 C CNN
+F 3 "~" H 3300 4700 50  0001 C CNN
+	1    3300 4700
+	1    0    0    -1
+$EndComp
+$Comp
+L Device:R R?
+U 1 1 605279D4
+P 3700 4700
+AR Path="/605279D4" Ref="R?"  Part="1"
+AR Path="/5F841BF9/605279D4" Ref="R?"  Part="1"
+AR Path="/5F8FEC08/605279D4" Ref="R?"  Part="1"
+F 0 "R?" H 3770 4746 50  0000 L CNN
+F 1 "330" H 3770 4655 50  0000 L CNN
+F 2 "Resistor_SMD:R_0603_1608Metric_Pad1.05x0.95mm_HandSolder" V 3630 4700 50  0001 C CNN
+F 3 "~" H 3700 4700 50  0001 C CNN
+	1    3700 4700
+	0    1    1    0
+$EndComp
+Text Notes 2900 4650 3    50   ~ 0
+BLU
+Wire Wire Line
+	3450 4700 3550 4700
+$Comp
+L power:GND #PWR?
+U 1 1 60527A35
+P 3100 5050
+AR Path="/60527A35" Ref="#PWR?"  Part="1"
+AR Path="/5F841BF9/60527A35" Ref="#PWR?"  Part="1"
+AR Path="/5F8FEC08/60527A35" Ref="#PWR?"  Part="1"
+F 0 "#PWR?" H 3100 4800 50  0001 C CNN
+F 1 "GND" H 3200 4950 50  0000 C CNN
+F 2 "" H 3100 5050 50  0001 C CNN
+F 3 "" H 3100 5050 50  0001 C CNN
+	1    3100 5050
+	0    1    1    0
+$EndComp
+$Comp
+L power:GND #PWR?
+U 1 1 60527A3B
+P 3100 4350
+AR Path="/60527A3B" Ref="#PWR?"  Part="1"
+AR Path="/5F841BF9/60527A3B" Ref="#PWR?"  Part="1"
+AR Path="/5F8FEC08/60527A3B" Ref="#PWR?"  Part="1"
+F 0 "#PWR?" H 3100 4100 50  0001 C CNN
+F 1 "GND" H 3200 4250 50  0000 C CNN
+F 2 "" H 3100 4350 50  0001 C CNN
+F 3 "" H 3100 4350 50  0001 C CNN
+	1    3100 4350
+	0    1    1    0
+$EndComp
+$Comp
+L power:GND #PWR?
+U 1 1 60527A41
+P 3100 4700
+AR Path="/60527A41" Ref="#PWR?"  Part="1"
+AR Path="/5F841BF9/60527A41" Ref="#PWR?"  Part="1"
+AR Path="/5F8FEC08/60527A41" Ref="#PWR?"  Part="1"
+F 0 "#PWR?" H 3100 4450 50  0001 C CNN
+F 1 "GND" H 3200 4600 50  0000 C CNN
+F 2 "" H 3100 4700 50  0001 C CNN
+F 3 "" H 3100 4700 50  0001 C CNN
+	1    3100 4700
+	0    1    1    0
+$EndComp
+Wire Wire Line
+	3100 4350 3150 4350
+Wire Wire Line
+	3100 4700 3150 4700
+Wire Wire Line
+	3100 5050 3150 5050
+Wire Wire Line
+	4300 4350 4300 4500
+Wire Wire Line
+	3850 4350 4300 4350
+Wire Wire Line
+	3850 4700 4200 4700
+Wire Wire Line
+	4300 5050 4300 4800
+Wire Wire Line
+	3850 5050 4225 5050
+Wire Wire Line
+	4200 4500 4300 4500
+Connection ~ 4300 4500
+Wire Wire Line
+	4300 4500 4300 4600
+Wire Wire Line
+	4200 4900 4200 4700
+Connection ~ 4200 4700
+Wire Wire Line
+	4200 4700 4400 4700
+Wire Wire Line
+	4225 5275 4225 5050
+Connection ~ 4225 5050
+Wire Wire Line
+	4225 5050 4300 5050
 $EndSCHEMATC

Commit message: Science_sensor reveiw 1
Yep
Parts:
- gave numbers to parts that had none: 7
Connections:
- net +5V: no longer names the net of U4.+5V (B1_1)
- net +5V: no longer U4.+5V (B2_1)
- no-connect marks 55 -> 57
Changed lines of the file:
@@
 	5300 4000 5450 4000
 $Comp
-L power:GND #PWR?
+L power:GND #PWR0166
 U 1 1 5F933A2E
 P 5450 4000
-F 0 "#PWR?" H 5450 3750 50  0001 C CNN
+F 0 "#PWR0166" H 5450 3750 50  0001 C CNN
 F 1 "GND" H 5455 3827 50  0000 C CNN
 F 2 "" H 5450 4000 50  0001 C CNN
@@
 	7200 2300 7200 2400
 $Comp
-L power:GND #PWR?
+L power:GND #PWR0167
 U 1 1 5F933A36
 P 7200 2300
-F 0 "#PWR?" H 7200 2050 50  0001 C CNN
+F 0 "#PWR0167" H 7200 2050 50  0001 C CNN
 F 1 "GND" H 7205 2127 50  0000 C CNN
 F 2 "" H 7200 2300 50  0001 C CNN
@@
 $EndComp
 $Comp
-L power:GND #PWR?
+L power:GND #PWR0168
 U 1 1 5F933A3C
 P 5950 2500
-F 0 "#PWR?" H 5950 2250 50  0001 C CNN
+F 0 "#PWR0168" H 5950 2250 50  0001 C CNN
 F 1 "GND" H 5955 2327 50  0000 C CNN
 F 2 "" H 5950 2500 50  0001 C CNN
@@
 	4300 2300 4300 2400
 $Comp
-L power:+3.3V #PWR?
+L power:+3.3V #PWR0169
 U 1 1 5F933A44
 P 4300 2300
-F 0 "#PWR?" H 4300 2150 50  0001 C CNN
+F 0 "#PWR0169" H 4300 2150 50  0001 C CNN
 F 1 "+3.3V" H 4315 2473 50  0000 C CNN
 F 2 "" H 4300 2300 50  0001 C CNN
@@
 NoConn ~ 7100 4300
 $Comp
-L power:+3.3V #PWR?
+L power:+3.3V #PWR0170
 U 1 1 5F933A79
 P 4300 3850
-F 0 "#PWR?" H 4300 3700 50  0001 C CNN
+F 0 "#PWR0170" H 4300 3700 50  0001 C CNN
 F 1 "+3.3V" H 4315 4023 50  0000 C CNN
 F 2 "" H 4300 3850 50  0001 C CNN
@@
 NoConn ~ 4400 2900
 $Comp
-L SRA_Sensor_Board-rescue:TM4C129E_Launchpad-MRDT_Shields-SRA_Sensor_Board-rescue U?
+L SRA_Sensor_Board-rescue:TM4C129E_Launchpad-MRDT_Shields-SRA_Sensor_Board-rescue U4
 U 4 1 5F933A8E
 P 6900 3350
-F 0 "U?" H 7000 3300 60  0000 C CNN
+F 0 "U4" H 7000 3300 60  0000 C CNN
 F 1 "TM4C129E_Launchpad" H 7150 3300 60  0001 C CNN
 F 2 "MRDT_Shields:TM4C129E_Launchpad_FULL_THT_BOTTOM" H 6900 3350 60  0001 C CNN
@@
 $EndComp
 $Comp
-L SRA_Sensor_Board-rescue:TM4C129E_Launchpad-MRDT_Shields-SRA_Sensor_Board-rescue U?
+L SRA_Sensor_Board-rescue:TM4C129E_Launchpad-MRDT_Shields-SRA_Sensor_Board-rescue U4
 U 3 1 5F933A94
 P 6400 3350
-F 0 "U?" H 6400 3300 60  0000 L CNN
+F 0 "U4" H 6400 3300 60  0000 L CNN
 F 1 "TM4C129E_Launchpad" H 6150 3300 60  0001 L CNN
 F 2 "MRDT_Shields:TM4C129E_Launchpad_FULL_THT_BOTTOM" H 6400 3350 60  0001 C CNN
@@
 $EndComp
 $Comp
-L SRA_Sensor_Board-rescue:TM4C129E_Launchpad-MRDT_Shields-SRA_Sensor_Board-rescue U?
+L SRA_Sensor_Board-rescue:TM4C129E_Launchpad-MRDT_Shields-SRA_Sensor_Board-rescue U4
 U 2 1 5F933A9A
 P 5100 3350
-F 0 "U?" H 5200 3300 60  0000 C CNN
+F 0 "U4" H 5200 3300 60  0000 C CNN
 F 1 "TM4C129E_Launchpad" H 5350 3300 60  0001 C CNN
 F 2 "MRDT_Shields:TM4C129E_Launchpad_FULL_THT_BOTTOM" H 5100 3350 60  0001 C CNN
@@
 $EndComp
 $Comp
-L SRA_Sensor_Board-rescue:TM4C129E_Launchpad-MRDT_Shields-SRA_Sensor_Board-rescue U?
+L SRA_Sensor_Board-rescue:TM4C129E_Launchpad-MRDT_Shields-SRA_Sensor_Board-rescue U4
 U 1 1 5F933AA0
 P 4600 3350
-F 0 "U?" H 4600 3300 60  0000 L CNN
+F 0 "U4" H 4600 3300 60  0000 L CNN
 F 1 "TM4C129E_Launchpad" H 4350 3300 60  0001 L CNN
 F 2 "MRDT_Shields:TM4C129E_Launchpad_FULL_THT_BOTTOM" H 4600 3350 60  0001 C CNN
@@
 	4300 3900 4400 3900
 $Comp
-L SRA_Sensor_Board-rescue:TM4C129E_Launchpad-MRDT_Shields U?
+L SRA_Sensor_Board-rescue:TM4C129E_Launchpad-MRDT_Shields U4
 U 5 1 5F933AAE
 P 4600 4850
-F 0 "U?" H 4600 4800 60  0000 L CNN
+F 0 "U4" H 4600 4800 60  0000 L CNN
 F 1 "TM4C129E_Launchpad" H 4400 4800 60  0001 L CNN
 F 2 "MRDT_Shields:TM4C129E_Launchpad_FULL_THT_BOTTOM" H 4600 4850 60  0001 C CNN
@@
 $EndComp
 $Comp
-L SRA_Sensor_Board-rescue:TM4C129E_Launchpad-MRDT_Shields U?
+L SRA_Sensor_Board-rescue:TM4C129E_Launchpad-MRDT_Shields U4
 U 6 1 5F933AB4
 P 5100 4850
-F 0 "U?" H 5200 4800 60  0000 C CNN
+F 0 "U4" H 5200 4800 60  0000 C CNN
 F 1 "TM4C129E_Launchpad" H 5300 4800 60  0001 C CNN
 F 2 "MRDT_Shields:TM4C129E_Launchpad_FULL_THT_BOTTOM" H 5100 4850 60  0001 C CNN
@@
 $EndComp
 Wire Wire Line
-	5400 3900 5300 3900
-Wire Wire Line
-	5400 3850 5400 3900
-$Comp
-L power:+5V #PWR?
-U 1 1 5F933ABC
-P 5400 3850
-F 0 "#PWR?" H 5400 3700 50  0001 C CNN
-F 1 "+5V" H 5415 4023 50  0000 C CNN
-F 2 "" H 5400 3850 50  0001 C CNN
-F 3 "" H 5400 3850 50  0001 C CNN
-	1    5400 3850
-	1    0    0    -1
-$EndComp
-Wire Wire Line
-	5400 2400 5300 2400
-Wire Wire Line
-	5400 2350 5400 2400
-$Comp
-L power:+5V #PWR?
-U 1 1 5F933AC4
-P 5400 2350
-F 0 "#PWR?" H 5400 2200 50  0001 C CNN
-F 1 "+5V" H 5415 2523 50  0000 C CNN
-F 2 "" H 5400 2350 50  0001 C CNN
-F 3 "" H 5400 2350 50  0001 C CNN
-	1    5400 2350
-	1    0    0    -1
-$EndComp
-Wire Wire Line
 	5300 2500 5950 2500
 Text GLabel 7150 2500 2    50   Output ~ 0
@@
 	7150 2500 7100 2500
 $Comp
-L SRA_Sensor_Board-rescue:TM4C129E_Launchpad-MRDT_Shields-SRA_Sensor_Board-rescue U?
+L SRA_Sensor_Board-rescue:TM4C129E_Launchpad-MRDT_Shields-SRA_Sensor_Board-rescue U4
 U 8 1 5F933ACF
 P 6900 4850
-F 0 "U?" H 7000 4800 60  0000 C CNN
+F 0 "U4" H 7000 4800 60  0000 C CNN
 F 1 "TM4C129E_Launchpad" H 7150 4800 60  0001 C CNN
 F 2 "MRDT_Shields:TM4C129E_Launchpad_FULL_THT_BOTTOM" H 6900 4850 60  0001 C CNN
@@
 $EndComp
 $Comp
-L SRA_Sensor_Board-rescue:TM4C129E_Launchpad-MRDT_Shields-SRA_Sensor_Board-rescue U?
+L SRA_Sensor_Board-rescue:TM4C129E_Launchpad-MRDT_Shields-SRA_Sensor_Board-rescue U4
 U 7 1 5F933AD5
 P 6400 4850
-F 0 "U?" H 6400 4800 60  0000 L CNN
+F 0 "U4" H 6400 4800 60  0000 L CNN
 F 1 "TM4C129E_Launchpad" H 6150 4800 60  0001 L CNN
 F 2 "MRDT_Shields:TM4C129E_Launchpad_FULL_THT_BOTTOM" H 6400 4850 60  0001 C CNN
@@
 NoConn ~ 6200 4000
 $Comp
-L power:GND #PWR?
+L power:GND #PWR0171
 U 1 1 5F933ADE
 P 7300 3900
-F 0 "#PWR?" H 7300 3650 50  0001 C CNN
+F 0 "#PWR0171" H 7300 3650 50  0001 C CNN
 F 1 "GND" H 7450 3850 50  0000 C CNN
 F 2 "" H 7300 3900 50  0001 C CNN
@@
 NoConn ~ 5300 2700
 NoConn ~ 5300 4600
-Text GLabel 4175 3325 0    50   Input ~ 0
+Text GLabel 4175 3325 0    50   Output ~ 0
 NO_SCL
 Text Notes 3775 3325 0    50   ~ 0
@@
 AR Path="/605279AE" Ref="D?"  Part="1"
 AR Path="/5F841BF9/605279AE" Ref="D?"  Part="1"
-AR Path="/5F8FEC08/605279AE" Ref="D?"  Part="1"
-F 0 "D?" V 3339 4933 50  0000 R CNN
+AR Path="/5F8FEC08/605279AE" Ref="D22"  Part="1"
+F 0 "D22" V 3339 4933 50  0000 R CNN
 F 1 "LED" V 3248 4933 50  0000 R CNN
 F 2 "Diode_SMD:D_0603_1608Metric_Pad1.05x0.95mm_HandSolder" H 3300 5050 50  0001 C CNN
@@
 AR Path="/605279B4" Ref="R?"  Part="1"
 AR Path="/5F841BF9/605279B4" Ref="R?"  Part="1"
-AR Path="/5F8FEC08/605279B4" Ref="R?"  Part="1"
-F 0 "R?" H 3770 5096 50  0000 L CNN
+AR Path="/5F8FEC08/605279B4" Ref="R40"  Part="1"
+F 0 "R40" H 3770 5096 50  0000 L CNN
 F 1 "330" H 3770 5005 50  0000 L CNN
 F 2 "Resistor_SMD:R_0603_1608Metric_Pad1.05x0.95mm_HandSolder" V 3630 5050 50  0001 C CNN
@@
 AR Path="/605279BE" Ref="D?"  Part="1"
 AR Path="/5F841BF9/605279BE" Ref="D?"  Part="1"
-AR Path="/5F8FEC08/605279BE" Ref="D?"  Part="1"
-F 0 "D?" V 3339 4233 50  0000 R CNN
+AR Path="/5F8FEC08/605279BE" Ref="D20"  Part="1"
+F 0 "D20" V 3339 4233 50  0000 R CNN
 F 1 "LED" V 3248 4233 50  0000 R CNN
 F 2 "Diode_SMD:D_0603_1608Metric_Pad1.05x0.95mm_HandSolder" H 3300 4350 50  0001 C CNN
@@
 AR Path="/605279C4" Ref="R?"  Part="1"
 AR Path="/5F841BF9/605279C4" Ref="R?"  Part="1"
-AR Path="/5F8FEC08/605279C4" Ref="R?"  Part="1"
-F 0 "R?" H 3770 4396 50  0000 L CNN
+AR Path="/5F8FEC08/605279C4" Ref="R38"  Part="1"
+F 0 "R38" H 3770 4396 50  0000 L CNN
 F 1 "330" H 3770 4305 50  0000 L CNN
 F 2 "Resistor_SMD:R_0603_1608Metric_Pad1.05x0.95mm_HandSolder" V 3630 4350 50  0001 C CNN
@@
 AR Path="/605279CE" Ref="D?"  Part="1"
 AR Path="/5F841BF9/605279CE" Ref="D?"  Part="1"
-AR Path="/5F8FEC08/605279CE" Ref="D?"  Part="1"
-F 0 "D?" V 3339 4583 50  0000 R CNN
+AR Path="/5F8FEC08/605279CE" Ref="D21"  Part="1"
+F 0 "D21" V 3339 4583 50  0000 R CNN
 F 1 "LED" V 3248 4583 50  0000 R CNN
 F 2 "Diode_SMD:D_0603_1608Metric_Pad1.05x0.95mm_HandSolder" H 3300 4700 50  0001 C CNN
@@
 AR Path="/605279D4" Ref="R?"  Part="1"
 AR Path="/5F841BF9/605279D4" Ref="R?"  Part="1"
-AR Path="/5F8FEC08/605279D4" Ref="R?"  Part="1"
-F 0 "R?" H 3770 4746 50  0000 L CNN
+AR Path="/5F8FEC08/605279D4" Ref="R39"  Part="1"
+F 0 "R39" H 3770 4746 50  0000 L CNN
 F 1 "330" H 3770 4655 50  0000 L CNN
 F 2 "Resistor_SMD:R_0603_1608Metric_Pad1.05x0.95mm_HandSolder" V 3630 4700 50  0001 C CNN
@@
 AR Path="/60527A35" Ref="#PWR?"  Part="1"
 AR Path="/5F841BF9/60527A35" Ref="#PWR?"  Part="1"
-AR Path="/5F8FEC08/60527A35" Ref="#PWR?"  Part="1"
-F 0 "#PWR?" H 3100 4800 50  0001 C CNN
+AR Path="/5F8FEC08/60527A35" Ref="#PWR0172"  Part="1"
+F 0 "#PWR0172" H 3100 4800 50  0001 C CNN
 F 1 "GND" H 3200 4950 50  0000 C CNN
 F 2 "" H 3100 5050 50  0001 C CNN
@@
 AR Path="/60527A3B" Ref="#PWR?"  Part="1"
 AR Path="/5F841BF9/60527A3B" Ref="#PWR?"  Part="1"
-AR Path="/5F8FEC08/60527A3B" Ref="#PWR?"  Part="1"
-F 0 "#PWR?" H 3100 4100 50  0001 C CNN
+AR Path="/5F8FEC08/60527A3B" Ref="#PWR0173"  Part="1"
+F 0 "#PWR0173" H 3100 4100 50  0001 C CNN
 F 1 "GND" H 3200 4250 50  0000 C CNN
 F 2 "" H 3100 4350 50  0001 C CNN
@@
 AR Path="/60527A41" Ref="#PWR?"  Part="1"
 AR Path="/5F841BF9/60527A41" Ref="#PWR?"  Part="1"
-AR Path="/5F8FEC08/60527A41" Ref="#PWR?"  Part="1"
-F 0 "#PWR?" H 3100 4450 50  0001 C CNN
+AR Path="/5F8FEC08/60527A41" Ref="#PWR0174"  Part="1"
+F 0 "#PWR0174" H 3100 4450 50  0001 C CNN
 F 1 "GND" H 3200 4600 50  0000 C CNN
 F 2 "" H 3100 4700 50  0001 C CNN
@@
 Wire Wire Line
 	4225 5050 4300 5050
+NoConn ~ 5300 2400
+NoConn ~ 5300 3900
 $EndSCHEMATC
