File: Hardware/SRASensorBoard_Hardware/TIVA.sch (KiCad schematic (older format))
At the start: 17 parts, among them U4 TM4C129E_Launchpad

Commit message: Finished BOM
Parts:
- D1, D2, D20, D21, D23, D3, D4: value LED -> Blue
- D22: value LED -> Red
Changed lines of the file:
@@
 AR Path="/5F8FEC08/605279AE" Ref="D22"  Part="1"
 F 0 "D22" V 3339 4933 50  0000 R CNN
-F 1 "LED" V 3248 4933 50  0000 R CNN
+F 1 "Red" V 3248 4933 50  0000 R CNN
 F 2 "Diode_SMD:D_0603_1608Metric_Pad1.05x0.95mm_HandSolder" H 3300 5050 50  0001 C CNN
 F 3 "~" H 3300 5050 50  0001 C CNN
@@
 AR Path="/5F8FEC08/605279BE" Ref="D20"  Part="1"
 F 0 "D20" V 3339 4233 50  0000 R CNN
-F 1 "LED" V 3248 4233 50  0000 R CNN
+F 1 "Blue" V 3248 4233 50  0000 R CNN
 F 2 "Diode_SMD:D_0603_1608Metric_Pad1.05x0.95mm_HandSolder" H 3300 4350 50  0001 C CNN
 F 3 "~" H 3300 4350 50  0001 C CNN
@@
 AR Path="/5F8FEC08/605279CE" Ref="D21"  Part="1"
 F 0 "D21" V 3339 4583 50  0000 R CNN
-F 1 "LED" V 3248 4583 50  0000 R CNN
+F 1 "Blue" V 3248 4583 50  0000 R CNN
 F 2 "Diode_SMD:D_0603_1608Metric_Pad1.05x0.95mm_HandSolder" H 3300 4700 50  0001 C CNN
 F 3 "~" H 3300 4700 50  0001 C CNN
@@
 AR Path="/5F8FEC08/60AEE3AC" Ref="D2"  Part="1"
 F 0 "D2" H 5750 2700 50  0000 R CNN
-F 1 "LED" H 5925 2700 50  0000 R CNN
+F 1 "Blue" H 5925 2700 50  0000 R CNN
 F 2 "Diode_SMD:D_0603_1608Metric_Pad1.05x0.95mm_HandSolder" H 6025 2650 50  0001 C CNN
 F 3 "~" H 6025 2650 50  0001 C CNN
@@
 AR Path="/5F8FEC08/60CF7541" Ref="D3"  Part="1"
 F 0 "D3" H 5750 2950 50  0000 R CNN
-F 1 "LED" H 5925 2950 50  0000 R CNN
+F 1 "Blue" H 5925 2950 50  0000 R CNN
 F 2 "Diode_SMD:D_0603_1608Metric_Pad1.05x0.95mm_HandSolder" H 6025 2900 50  0001 C CNN
 F 3 "~" H 6025 2900 50  0001 C CNN
@@
 AR Path="/5F8FEC08/60D61465" Ref="D4"  Part="1"
 F 0 "D4" H 5775 3225 50  0000 R CNN
-F 1 "LED" H 5950 3225 50  0000 R CNN
+F 1 "Blue" H 5950 3225 50  0000 R CNN
 F 2 "Diode_SMD:D_0603_1608Metric_Pad1.05x0.95mm_HandSolder" H 6050 3175 50  0001 C CNN
 F 3 "~" H 6050 3175 50  0001 C CNN
@@
 AR Path="/5F8FEC08/60E141AA" Ref="D23"  Part="1"
 F 0 "D23" H 5775 3475 50  0000 R CNN
-F 1 "LED" H 5950 3475 50  0000 R CNN
+F 1 "Blue" H 5950 3475 50  0000 R CNN
 F 2 "Diode_SMD:D_0603_1608Metric_Pad1.05x0.95mm_HandSolder" H 6050 3425 50  0001 C CNN
 F 3 "~" H 6050 3425 50  0001 C CNN
@@
 AR Path="/5F8FEC08/60EBE8F2" Ref="D1"  Part="1"
 F 0 "D1" H 3625 4025 50  0000 R CNN
-F 1 "LED" H 3500 4025 50  0000 R CNN
+F 1 "Blue" H 3500 4025 50  0000 R CNN
 F 2 "Diode_SMD:D_0603_1608Metric_Pad1.05x0.95mm_HandSolder" H 3600 3925 50  0001 C CNN
 F 3 "~" H 3600 3925 50  0001 C CNN
