File: Hardware/SRASensorBoard_Hardware/POWER.sch (KiCad schematic (older format))
At the start: 16 parts

Commit message: Sciency stuff for the board
finished!
Parts:
- added D? (x4): LED, Diode_SMD:D_0603_1608Metric_Pad1.05x0.95mm_HandSolder, symbol Device:LED
- added R?: 510, Resistor_SMD:R_0603_1608Metric_Pad1.05x0.95mm_HandSolder, symbol Device:R
- added R?: 330, Resistor_SMD:R_0603_1608Metric_Pad1.05x0.95mm_HandSolder, symbol Device:R
- added R?: 1000, Resistor_SMD:R_0603_1608Metric_Pad1.05x0.95mm_HandSolder, symbol Device:R
- added R?: 2500, Resistor_SMD:R_0603_1608Metric_Pad1.05x0.95mm_HandSolder, symbol Device:R
Connections:
- wire segments 35 -> 47
Other:
- note added: "GREEN"
- moved on the sheet: C?, Conn?A, Conn?B

Commit message: Science_sensor reveiw 1
Yep
Parts:
- C1, C2: renamed from C?; footprint (none) -> Capacitor_SMD:C_0603_1608Metric
- C3, C4: renamed from C?; footprint (none) -> Capacitor_THT:CP_Radial_D10.0mm_P5.00mm
- D1, D2: renamed from D?; footprint (none) -> Diode_SMD:D_0603_1608Metric
- L1, L2: renamed from L?; footprint (none) -> Inductor_SMD:L_0201_0603Metric
- U1, U2: renamed from U?; footprint Package_TO_SOT_SMD:TO-263-5_TabPin3 -> MRDT_Devices:LM2576
- gave numbers to parts that had none: 11

Commit message: Layout started, edge cut fix
ladybug is not pleased
Parts:
- removed D1, D2: 1N5822, Diode_SMD:D_0603_1608Metric, symbol Device:D_Schottky
- removed D3, D4: LED, Diode_SMD:D_0603_1608Metric_Pad1.05x0.95mm_HandSolder, symbol Device:LED
- removed L1, L2: 100uH, Inductor_SMD:L_0201_0603Metric, symbol Device:L
- removed R1: 330, Resistor_SMD:R_0603_1608Metric_Pad1.05x0.95mm_HandSolder, symbol Device:R
- removed R2: 510, Resistor_SMD:R_0603_1608Metric_Pad1.05x0.95mm_HandSolder, symbol Device:R
- removed U1: LM2576S-3.3, MRDT_Devices:LM2576, symbol Regulator_Switching:LM2576S-3.3
- removed U2: LM2576HVS-5, MRDT_Devices:LM2576, symbol Regulator_Switching:LM2576HVS-5
- added unit 3 of Conn1
- added U1, U2: OKI, MRDT_Devices:OKI_Horizontal, symbol MRDT_Devices:OKI
- C1, C2: value 100uF -> 10uF; footprint Capacitor_SMD:C_0603_1608Metric -> Capacitor_SMD:C_0603_1608Metric_Pad1.05x0.95mm_HandSolder
- C3, C4: value 1000uF -> 10uF; footprint Capacitor_THT:CP_Radial_D10.0mm_P5.00mm -> Capacitor_SMD:C_0603_1608Metric_Pad1.05x0.95mm_HandSolder
- Conn1: footprint MRDT_Connectors:Anderson_2_Horizontal_Side_by_Side -> MRDT_Connectors:Anderson_3_Horizontal_Side_by_Side
Connections:
- net labels added: +12VA
- wire segments 47 -> 40
Other:
- moved on the sheet: C1, Conn1B

Commit message: Fixed some library issues
Parts:
- C1, C2, C3, C4: footprint Capacitor_SMD:C_0603_1608Metric_Pad1.05x0.95mm_HandSolder -> Capacitor_SMD:C_0603_1608Metric_Pad1.08x0.95mm_HandSolder
- R3: value 1000 -> 1K; footprint Resistor_SMD:R_0603_1608Metric_Pad1.05x0.95mm_HandSolder -> Resistor_SMD:R_0603_1608Metric_Pad0.98x0.95mm_HandSolder
- R4: value 2500 -> 2.5K; footprint Resistor_SMD:R_0603_1608Metric_Pad1.05x0.95mm_HandSolder -> Resistor_SMD:R_0603_1608Metric_Pad0.98x0.95mm_HandSolder
Changed lines of the file:
@@
 EESchema Schematic File Version 4
+LIBS:SRA_Sensor_Board-cache
 EELAYER 30 0
 EELAYER END
@@
 F 0 "C1" H 3090 2871 50  0000 L CNN
 F 1 "10uF" H 3090 2780 50  0000 L CNN
-F 2 "Capacitor_SMD:C_0603_1608Metric_Pad1.05x0.95mm_HandSolder" H 3013 2675 50  0001 C CNN
+F 2 "Capacitor_SMD:C_0603_1608Metric_Pad1.08x0.95mm_HandSolder" H 3013 2675 50  0001 C CNN
 F 3 "~" H 2975 2825 50  0001 C CNN
 	1    2975 2825
@@
 F 0 "C2" H 3165 4271 50  0000 L CNN
 F 1 "10uF" H 3165 4180 50  0000 L CNN
-F 2 "Capacitor_SMD:C_0603_1608Metric_Pad1.05x0.95mm_HandSolder" H 3088 4075 50  0001 C CNN
+F 2 "Capacitor_SMD:C_0603_1608Metric_Pad1.08x0.95mm_HandSolder" H 3088 4075 50  0001 C CNN
 F 3 "~" H 3050 4225 50  0001 C CNN
 	1    3050 4225
@@
 AR Path="/5F7D791F/6057C1C6" Ref="R3"  Part="1"
 F 0 "R3" H 8720 2971 50  0000 L CNN
-F 1 "1000" H 8720 2880 50  0000 L CNN
-F 2 "Resistor_SMD:R_0603_1608Metric_Pad1.05x0.95mm_HandSolder" V 8580 2925 50  0001 C CNN
+F 1 "1K" H 8720 2880 50  0000 L CNN
+F 2 "Resistor_SMD:R_0603_1608Metric_Pad0.98x0.95mm_HandSolder" V 8580 2925 50  0001 C CNN
 F 3 "~" H 8650 2925 50  0001 C CNN
 	1    8650 2925
@@
 AR Path="/5F7D791F/6057C22C" Ref="R4"  Part="1"
 F 0 "R4" H 8720 3421 50  0000 L CNN
-F 1 "2500" H 8720 3330 50  0000 L CNN
-F 2 "Resistor_SMD:R_0603_1608Metric_Pad1.05x0.95mm_HandSolder" V 8580 3375 50  0001 C CNN
+F 1 "2.5K" H 8720 3330 50  0000 L CNN
+F 2 "Resistor_SMD:R_0603_1608Metric_Pad0.98x0.95mm_HandSolder" V 8580 3375 50  0001 C CNN
 F 3 "~" H 8650 3375 50  0001 C CNN
 	1    8650 3375
@@
 F 0 "C4" H 4515 3071 50  0000 L CNN
 F 1 "10uF" H 4515 2980 50  0000 L CNN
-F 2 "Capacitor_SMD:C_0603_1608Metric_Pad1.05x0.95mm_HandSolder" H 4438 2875 50  0001 C CNN
+F 2 "Capacitor_SMD:C_0603_1608Metric_Pad1.08x0.95mm_HandSolder" H 4438 2875 50  0001 C CNN
 F 3 "~" H 4400 3025 50  0001 C CNN
 	1    4400 3025
@@
 F 0 "C3" H 4440 4471 50  0000 L CNN
 F 1 "10uF" H 4440 4380 50  0000 L CNN
-F 2 "Capacitor_SMD:C_0603_1608Metric_Pad1.05x0.95mm_HandSolder" H 4363 4275 50  0001 C CNN
+F 2 "Capacitor_SMD:C_0603_1608Metric_Pad1.08x0.95mm_HandSolder" H 4363 4275 50  0001 C CNN
 F 3 "~" H 4325 4425 50  0001 C CNN
 	1    4325 4425

Commit message: Finished BOM
Parts:
- D5, D6: value LED -> Green
Changed lines of the file:
@@
 AR Path="/5F7D791F/6057C17D" Ref="D6"  Part="1"
 F 0 "D6" V 9089 3258 50  0000 R CNN
-F 1 "LED" V 8998 3258 50  0000 R CNN
+F 1 "Green" V 8998 3258 50  0000 R CNN
 F 2 "Diode_SMD:D_0603_1608Metric_Pad1.05x0.95mm_HandSolder" H 9050 3375 50  0001 C CNN
 F 3 "~" H 9050 3375 50  0001 C CNN
@@
 AR Path="/5F7D791F/6057C1C0" Ref="D5"  Part="1"
 F 0 "D5" V 9089 2808 50  0000 R CNN
-F 1 "LED" V 8998 2808 50  0000 R CNN
+F 1 "Green" V 8998 2808 50  0000 R CNN
 F 2 "Diode_SMD:D_0603_1608Metric_Pad1.05x0.95mm_HandSolder" H 9050 2925 50  0001 C CNN
 F 3 "~" H 9050 2925 50  0001 C CNN
