File: Hardware/SRASensorBoard_Hardware/sensors.sch (KiCad schematic (older format))
At the start: 57 parts, among them J1 USB_A, Q2 BSS138, Q3 BSS138, Q4 BSS138, Q5 BSS138, Q6 BSS138, U4 FT230XS

Commit message: Started Rev 2, NO sensor schematic
Parts:
- removed Conn2: Molex_SL_03, MRDT_Connectors:MOLEX_SL_03_Horizontal, symbol MRDT_Connectors:Molex_SL_03
- added C11, C13: 2.2uF, symbol Device:C
- added C12, C14: 3.3nF, symbol Device:C
- added Conn2: Molex_SL_04, MRDT_Connectors:MOLEX_SL_04_Horizontal, symbol MRDT_Connectors:Molex_SL_04
- added D20: Blue, LED_SMD:LED_0603_1608Metric_Pad1.05x0.95mm_HandSolder, symbol Device:LED
- added R44, R45: 240, Resistor_SMD:R_0603_1608Metric_Pad1.05x0.95mm_HandSolder, symbol Device:R
- added R46, R48: 56k, symbol Device:R
- added R47, R49: 1M, symbol Device:R
- added U5, U6: TSV911RILT, Package_TO_SOT_SMD:SOT-23-5, symbol Amplifier_Operational:TSV911RILT
Connections:
- net labels added: NO_Gas
- net labels removed: +12V
- wire segments 200 -> 245
Other:
- note added: "NO_Sensor"
- note removed: "NH3_Breakout"
- moved on the sheet: D6, Q2, Q3, Q4, Q5, Q6, R15, R16, R18, R19, R22, R23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

Commit message: added NO sensor stuff and finished layout
Parts:
- C11, C12, C13, C14: footprint (none) -> Capacitor_SMD:C_0603_1608Metric_Pad1.08x0.95mm_HandSolder
- R46, R47, R48, R49: footprint (none) -> Resistor_SMD:R_0603_1608Metric_Pad0.98x0.95mm_HandSolder
Changed lines of the file:
@@
 F 0 "R49" V 3550 6450 50  0000 C CNN
 F 1 "1M" V 3650 6450 50  0000 C CNN
-F 2 "" V 3580 6450 50  0001 C CNN
+F 2 "Resistor_SMD:R_0603_1608Metric_Pad0.98x0.95mm_HandSolder" V 3580 6450 50  0001 C CNN
 F 3 "~" H 3650 6450 50  0001 C CNN
 	1    3650 6450
@@
 F 0 "C14" V 3398 6900 50  0000 C CNN
 F 1 "3.3nF" V 3489 6900 50  0000 C CNN
-F 2 "" H 3688 6750 50  0001 C CNN
+F 2 "Capacitor_SMD:C_0603_1608Metric_Pad1.08x0.95mm_HandSolder" H 3688 6750 50  0001 C CNN
 F 3 "~" H 3650 6900 50  0001 C CNN
 	1    3650 6900
@@
 F 0 "C13" V 3023 6225 50  0000 C CNN
 F 1 "2.2uF" V 3114 6225 50  0000 C CNN
-F 2 "" H 3313 6075 50  0001 C CNN
+F 2 "Capacitor_SMD:C_0603_1608Metric_Pad1.08x0.95mm_HandSolder" H 3313 6075 50  0001 C CNN
 F 3 "~" H 3275 6225 50  0001 C CNN
 	1    3275 6225
@@
 F 0 "R48" V 3550 6225 50  0000 C CNN
 F 1 "56k" V 3650 6225 50  0000 C CNN
-F 2 "" V 3580 6225 50  0001 C CNN
+F 2 "Resistor_SMD:R_0603_1608Metric_Pad0.98x0.95mm_HandSolder" V 3580 6225 50  0001 C CNN
 F 3 "~" H 3650 6225 50  0001 C CNN
 	1    3650 6225
@@
 F 0 "R47" V 1600 6475 50  0000 C CNN
 F 1 "1M" V 1700 6475 50  0000 C CNN
-F 2 "" V 1630 6475 50  0001 C CNN
+F 2 "Resistor_SMD:R_0603_1608Metric_Pad0.98x0.95mm_HandSolder" V 1630 6475 50  0001 C CNN
 F 3 "~" H 1700 6475 50  0001 C CNN
 	1    1700 6475
@@
 F 0 "C12" V 1448 6925 50  0000 C CNN
 F 1 "3.3nF" V 1539 6925 50  0000 C CNN
-F 2 "" H 1738 6775 50  0001 C CNN
+F 2 "Capacitor_SMD:C_0603_1608Metric_Pad1.08x0.95mm_HandSolder" H 1738 6775 50  0001 C CNN
 F 3 "~" H 1700 6925 50  0001 C CNN
 	1    1700 6925
@@
 F 0 "C11" V 1073 6250 50  0000 C CNN
 F 1 "2.2uF" V 1164 6250 50  0000 C CNN
-F 2 "" H 1363 6100 50  0001 C CNN
+F 2 "Capacitor_SMD:C_0603_1608Metric_Pad1.08x0.95mm_HandSolder" H 1363 6100 50  0001 C CNN
 F 3 "~" H 1325 6250 50  0001 C CNN
 	1    1325 6250
@@
 F 0 "R46" V 1600 6250 50  0000 C CNN
 F 1 "56k" V 1700 6250 50  0000 C CNN
-F 2 "" V 1630 6250 50  0001 C CNN
+F 2 "Resistor_SMD:R_0603_1608Metric_Pad0.98x0.95mm_HandSolder" V 1630 6250 50  0001 C CNN
 F 3 "~" H 1700 6250 50  0001 C CNN
 	1    1700 6250
