File: Hardware/SRASensorBoard_Hardware/sensors.sch (KiCad schematic (older format))
At the start: 55 parts, among them J1 USB_A, Q1 BSS138, Q10 BSS138, Q11 BSS138, Q2 BSS138, Q3 BSS138, Q4 BSS138, Q5 BSS138, Q6 BSS138, U4 FT230XS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

Commit message: added teensy
Parts:
- C10, C5, C6, C7: footprint Capacitor_SMD:C_0603_1608Metric_Pad1.05x0.95mm_HandSolder -> Capacitor_SMD:C_0603_1608Metric_Pad1.08x0.95mm_HandSolder
- FB1: footprint Resistor_SMD:R_0805_2012Metric_Pad1.15x1.40mm_HandSolder -> Capacitor_SMD:C_0603_1608Metric_Pad1.08x0.95mm_HandSolder
Changed lines of the file:
@@
 F 0 "FB1" V 4425 1850 50  0000 C CNN
 F 1 "Ferrite_Bead" V 4700 1900 50  0000 C CNN
-F 2 "Resistor_SMD:R_0805_2012Metric_Pad1.15x1.40mm_HandSolder" V 4505 1825 50  0001 C CNN
+F 2 "Capacitor_SMD:C_0603_1608Metric_Pad1.08x0.95mm_HandSolder" V 4505 1825 50  0001 C CNN
 F 3 "~" H 4575 1825 50  0001 C CNN
 	1    4575 1825
@@
 F 0 "C5" V 3973 1525 50  0000 C CNN
 F 1 "10nF" V 4064 1525 50  0000 C CNN
-F 2 "Capacitor_SMD:C_0603_1608Metric_Pad1.05x0.95mm_HandSolder" H 4263 1375 50  0001 C CNN
+F 2 "Capacitor_SMD:C_0603_1608Metric_Pad1.08x0.95mm_HandSolder" H 4263 1375 50  0001 C CNN
 F 3 "~" H 4225 1525 50  0001 C CNN
 	1    4225 1525
@@
 F 0 "C10" V 6352 2950 50  0000 C CNN
 F 1 "100nF" V 6261 2950 50  0000 C CNN
-F 2 "Capacitor_SMD:C_0603_1608Metric_Pad1.05x0.95mm_HandSolder" H 6138 2800 50  0001 C CNN
+F 2 "Capacitor_SMD:C_0603_1608Metric_Pad1.08x0.95mm_HandSolder" H 6138 2800 50  0001 C CNN
 F 3 "~" H 6100 2950 50  0001 C CNN
 	1    6100 2950
@@
 F 0 "C6" V 4250 1100 50  0000 L CNN
 F 1 "100nF" V 4325 1150 50  0000 L CNN
-F 2 "Capacitor_SMD:C_0603_1608Metric_Pad1.05x0.95mm_HandSolder" H 4513 1100 50  0001 C CNN
+F 2 "Capacitor_SMD:C_0603_1608Metric_Pad1.08x0.95mm_HandSolder" H 4513 1100 50  0001 C CNN
 F 3 "~" H 4475 1250 50  0001 C CNN
 	1    4475 1250
@@
 F 0 "C7" V 4675 1350 50  0000 C CNN
 F 1 "4.7 uF" V 4600 1450 50  0000 C CNN
-F 2 "Capacitor_SMD:C_0603_1608Metric_Pad1.05x0.95mm_HandSolder" H 4475 1450 50  0001 C CNN
+F 2 "Capacitor_SMD:C_0603_1608Metric_Pad1.08x0.95mm_HandSolder" H 4475 1450 50  0001 C CNN
 F 3 "~" H 4475 1450 50  0001 C CNN
 	1    4475 1450
