File: Hardware/SRASensorBoard_Hardware/SRA_Sensor_Board.kicad_pcb (KiCad board)
At the start: 2 copper layers, 76.2 x 127 mm, 90 parts, among them J1 USB_A, Q2 BSS138, Q3 BSS138, Q4 BSS138, Q5 BSS138, Q6 BSS138, Q7 BSS214NW, Q8 BSS214NW, Q9 BSS214NW, U2 TSR1-2433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

Commit message: worked on layout
Parts:
- removed C1, C2, C3, C4: 10uf, Capacitor_SMD:C_0603_1608Metric_Pad1.08x0.95mm_HandSolder
- removed C10, C6: 100nF, Capacitor_SMD:C_0603_1608Metric_Pad1.08x0.95mm_HandSolder
- removed C11, C13: 2.2uF, Capacitor_SMD:C_0603_1608Metric_Pad1.08x0.95mm_HandSolder
- removed C12, C14: 3.3nF, Capacitor_SMD:C_0603_1608Metric_Pad1.08x0.95mm_HandSolder
- removed C5: 10nF, Capacitor_SMD:C_0603_1608Metric_Pad1.08x0.95mm_HandSolder
- removed C7: 4.7 uF, Capacitor_SMD:C_0603_1608Metric_Pad1.08x0.95mm_HandSolder
- removed C8, C9: 47pF, Capacitor_SMD:C_01005_0402Metric
- removed Conn1: AndersonPP, MRDT_Connectors:Anderson_2_Horizontal_Side_by_Side
- removed Conn10, Conn11, Conn12, Conn13, Conn14, Conn7, Conn8, Conn9: Molex_SL_02, MRDT_Connectors:MOLEX_SL_02_Horizontal
- removed Conn2, Conn4, Conn5: Molex_SL_04, MRDT_Connectors:MOLEX_SL_04_Horizontal
- removed D1, D2: Green, LED_SMD:LED_0603_1608Metric_Pad1.05x0.95mm_HandSolder
- removed D14, D15, D16, D17, D18, D19, D3, D4, D5, D9: Blue, LED_SMD:LED_0603_1608Metric_Pad1.05x0.95mm_HandSolder
- removed FB1: Ferrite_Bead, Capacitor_SMD:C_0603_1608Metric_Pad1.08x0.95mm_HandSolder
- removed J1: USB_A, Connector_USB:USB_A_Stewart_SS-52100-001_Horizontal
- removed Q2, Q3, Q4, Q5, Q6: BSS138, Package_TO_SOT_SMD:SOT-23
- removed Q7, Q8, Q9: BSS214NW, Package_TO_SOT_SMD:SOT-323_SC-70
- removed R1: 300, Resistor_SMD:R_0603_1608Metric_Pad0.98x0.95mm_HandSolder
- removed R15, R16, R18, R19, R22, R23, R24, R25, R26, R27: 10K, Resistor_SMD:R_0603_1608Metric_Pad0.98x0.95mm_HandSolder
- removed R17, R28, R29, R31, R36, R37, R38, R39, R40, R41, R5: 330, Resistor_SMD:R_0603_1608Metric_Pad0.98x0.95mm_HandSolder
- removed R2, R3, R4, R42, R43: 130, Resistor_SMD:R_0603_1608Metric_Pad0.98x0.95mm_HandSolder
- removed R20, R21: 27, Resistor_SMD:R_0603_1608Metric_Pad0.98x0.95mm_HandSolder
- removed R46, R48: 56k, Resistor_SMD:R_0603_1608Metric_Pad0.98x0.95mm_HandSolder
- removed R47, R49: 1M, Resistor_SMD:R_0603_1608Metric_Pad0.98x0.95mm_HandSolder
- removed U2: TSR1-2433, MRDT_Devices:TSR_1-2433
- removed U4: FT230XS, Package_SO:SSOP-16_3.9x4.9mm_P0.635mm
- removed U5, U6: TSV911RILT, Package_TO_SOT_SMD:SOT-23-5
- removed V1, V2, V3, V4: Via, MRDT_Drill_Holes:4_40_Hole_Corner
- moved U3 4.83 mm to (120.1, 67.6)
Routing:
- net O2_TX: track 0.00 -> 112.0 mm, vias 0 -> 1
- net O2_RX: track 0.00 -> 105.3 mm, vias 0 -> 1
- net Net-(Conn2-Pad3): track 0.00 -> 75.5 mm, vias 0 -> 4
- net NO2_CS: track 0.00 -> 69.2 mm, vias 0 -> 2
- net NO2_SCK: track 0.00 -> 67.6 mm, vias 0 -> 2
- net NO2_MISO: track 0.00 -> 64.6 mm, vias 0 -> 2
- net Net-(Conn2-Pad2): track 0.00 -> 62.2 mm, vias 0 -> 2
- net Net-(Conn7-Pad1): track 62.3 -> 3.42 mm, vias 3 -> 1
- net UVLED: track 57.3 -> 1.25 mm, vias 2 -> 1
- net Lights: track 49.9 -> 1.25 mm, vias 2 -> 1
- net Net-(Conn9-Pad1): track 46.0 -> 3.17 mm, vias 3 -> 1
- net Photodiode3: track 30.6 -> 0.00 mm
- net NO2_MISO_TIVA: track 0.00 -> 29.1 mm, vias 0 -> 2
- net NO2_CS_TIVA: track 1.82 -> 29.3 mm, vias 1 -> 2
- net TIVA_O2_TX: track 2.18 -> 28.7 mm, vias 1 -> 2
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
Commit message: finished layout
Routing:
- net +5V: track 0.00 -> 409.9 mm, vias 0 -> 35
- net +3V3: track 10.5 -> 329.6 mm, vias 0 -> 13
- net Photodiode2: track 0.18 -> 131.9 mm, vias 0 -> 4
- net +12V: track 0.00 -> 112.8 mm, vias 0 -> 5
- net Photodiode1: track 0.00 -> 105.7 mm, vias 0 -> 4
- net Net-(Conn9-Pad1): track 3.17 -> 91.3 mm, vias 1 -> 5
- net CH4_RX: track 0.00 -> 76.0 mm, vias 0 -> 4
- net CH4_TX: track 0.00 -> 74.8 mm, vias 0 -> 4
- net Net-(Conn7-Pad1): track 3.42 -> 67.9 mm, vias 1 -> 4
- net Net-(Conn11-Pad1): track 3.42 -> 62.0 mm, vias 1 -> 5
- net UVLED: track 1.25 -> 52.3 mm, vias 1 -> 3
- net Photodiode3: track 0.00 -> 48.8 mm, vias 0 -> 2
- net Lights: track 1.25 -> 45.1 mm, vias 1 -> 3
- net Net-(C10-Pad1): track 0.00 -> 24.9 mm, vias 0 -> 4
- net /Sheet615E4949/D2+: track 0.00 -> 8.43 mm
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