File: Hardware/ScienceSensor/Lasers & Photodiode.sch (KiCad schematic (older format))
At the start: 0 parts

Commit message: Lasers
Parts:
- added Conn? (x3): Molex_SL_02, symbol MRDT_Connectors:Molex_SL_02
- added D? (x3): LED, symbol Device:LED
- added Q? (x3): BSS214NW, Package_TO_SOT_SMD:SOT-323_SC-70, symbol Transistor_FET:BSS214NW
- added R? (x3): R, symbol Device:R
Connections:
- new net: Conn?.1, Q?.2 (S), R?.1 (x3)
- new net: D?.2 (A), R?.2 (x3)
- new net +12V: Q?.3 (D), Q?.3 (D), Q?.3 (D)
- new net GND: Conn?.2, Conn?.2, Conn?.2, D?.1 (K), D?.1 (K), D?.1 (K)
- new net Laser_1: Q?.1 (G)
- new net Laser_2: Q?.1 (G)
- new net Laser_3: Q?.1 (G)
Other:
- note added: "Laser 1"
- note added: "Laser 2"
- note added: "Laser 3"
