File: Hardware/ScienceSensor/Teensy.kicad_sch (KiCad schematic)
At the start: 10 parts, among them J2 6P6C, J3 RJ45_LED_Shielded, U3 Teensy4.1_DEV-16771

Commit message: Schematic Review
Parts:
- removed D3, D4, D5: Blue, symbol Device:LED
- removed R3, R4, R5: 130, symbol Device:R
Connections:
- no-connect marks 38 -> 41
Changed lines of the file:
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@@
   (no_connect (at 70.485 81.28))
   (no_connect (at 70.485 78.74))
+  (no_connect (at 70.485 127))
+  (no_connect (at 70.485 129.54))
   (no_connect (at 111.125 55.88))
   (no_connect (at 111.125 53.34))
@@
   (no_connect (at 111.125 48.26))
   (no_connect (at 70.485 99.06))
+  (no_connect (at 70.485 124.46))
   (no_connect (at 111.125 78.74))
   (no_connect (at 111.125 58.42))
@@
   (no_connect (at 70.485 55.88))
   (no_connect (at 111.125 71.12))
-  (wire (pts (xy 55.245 141.605) (xy 55.245 143.51))
-    (stroke (width 0) (type default) (color 0 0 0 0))
-  )
   (wire (pts (xy 207.01 40.005) (xy 197.485 40.005))
     (stroke (width 0) (type default) (color 0 0 0 0))
@@
     (stroke (width 0) (type default) (color 0 0 0 0))
   )
-  (wire (pts (xy 70.485 127) (xy 60.96 127))
-    (stroke (width 0) (type default) (color 0 0 0 0))
-  )
   (wire (pts (xy 118.745 134.62) (xy 118.745 137.16))
     (stroke (width 0) (type default) (color 0 0 0 0))
@@
     (stroke (width 0) (type default) (color 0 0 0 0))
   )
-  (wire (pts (xy 60.96 135.255) (xy 60.96 140.97))
-    (stroke (width 0) (type default) (color 0 0 0 0))
-  )
   (wire (pts (xy 66.675 76.2) (xy 70.485 76.2))
     (stroke (width 0) (type default) (color 0 0 0 0))
@@
     (stroke (width 0) (type default) (color 0 0 0 0))
   )
-  (wire (pts (xy 55.245 124.46) (xy 55.245 125.095))
-    (stroke (width 0) (type default) (color 0 0 0 0))
-  )
   (wire (pts (xy 189.865 62.865) (xy 189.865 66.675))
     (stroke (width 0) (type default) (color 0 0 0 0))
@@
     (stroke (width 0) (type default) (color 0 0 0 0))
   )
-  (wire (pts (xy 66.675 155.575) (xy 66.675 157.48))
-    (stroke (width 0) (type default) (color 0 0 0 0))
-  )
   (wire (pts (xy 70.485 111.76) (xy 64.135 111.76))
     (stroke (width 0) (type default) (color 0 0 0 0))
@@
     (stroke (width 0) (type default) (color 0 0 0 0))
   )
-  (wire (pts (xy 70.485 124.46) (xy 55.245 124.46))
-    (stroke (width 0) (type default) (color 0 0 0 0))
-  )
   (wire (pts (xy 189.865 77.47) (xy 207.01 77.47))
     (stroke (width 0) (type default) (color 0 0 0 0))
@@
     (stroke (width 0) (type default) (color 0 0 0 0))
   )
-  (wire (pts (xy 60.96 127) (xy 60.96 127.635))
-    (stroke (width 0) (type default) (color 0 0 0 0))
-  )
   (wire (pts (xy 70.485 104.14) (xy 64.135 104.14))
     (stroke (width 0) (type default) (color 0 0 0 0))
@@
     (stroke (width 0) (type default) (color 0 0 0 0))
   )
-  (wire (pts (xy 70.485 129.54) (xy 66.675 129.54))
-    (stroke (width 0) (type default) (color 0 0 0 0))
-  )
   (wire (pts (xy 70.485 68.58) (xy 66.675 68.58))
     (stroke (width 0) (type default) (color 0 0 0 0))
@@
     (stroke (width 0) (type default) (color 0 0 0 0))
   )
-  (wire (pts (xy 55.245 132.715) (xy 55.245 133.985))
-    (stroke (width 0) (type default) (color 0 0 0 0))
-  )
   (wire (pts (xy 192.405 66.04) (xy 192.405 64.77))
     (stroke (width 0) (type default) (color 0 0 0 0))
@@
     (stroke (width 0) (type default) (color 0 0 0 0))
   )
-  (wire (pts (xy 60.96 148.59) (xy 60.96 150.495))
-    (stroke (width 0) (type default) (color 0 0 0 0))
-  )
   (wire (pts (xy 194.945 66.675) (xy 194.945 80.01))
     (stroke (width 0) (type default) (color 0 0 0 0))
@@
     (stroke (width 0) (type default) (color 0 0 0 0))
   )
-  (wire (pts (xy 66.675 129.54) (xy 66.675 131.445))
-    (stroke (width 0) (type default) (color 0 0 0 0))
-  )
   (wire (pts (xy 207.01 77.47) (xy 207.01 40.005))
     (stroke (width 0) (type default) (color 0 0 0 0))
@@
   )
   (wire (pts (xy 197.485 40.005) (xy 197.485 42.545))
-    (stroke (width 0) (type default) (color 0 0 0 0))
-  )
-  (wire (pts (xy 66.675 139.065) (xy 66.675 147.955))
     (stroke (width 0) (type default) (color 0 0 0 0))
   )
@@
     (pin "VUSB")
   )
-  (symbol (lib_id "Device:R") (at 66.675 135.255 0) (unit 1)
-    (in_bom yes) (on_board yes)
-    (property "Reference" "R5" (id 0) (at 68.453 134.0866 0)
-      (effects (font (size 1.27 1.27)) (justify left))
-    )
-    (property "Value" "130" (id 1) (at 66.675 137.16 90)
-      (effects (font (size 1.27 1.27)) (justify left))
-    )
-    (property "Footprint" "" (id 2) (at 64.897 135.255 90)
-      (effects (font (size 1.27 1.27)) hide)
-    )
-    (property "Datasheet" "~" (id 3) (at 66.675 135.255 0)
-      (effects (font (size 1.27 1.27)) hide)
-    )
-    (pin "1")
-    (pin "2")
-  )
-  (symbol (lib_id "Device:R") (at 60.96 131.445 0) (unit 1)
-    (in_bom yes) (on_board yes)
-    (property "Reference" "R4" (id 0) (at 62.738 130.2766 0)
-      (effects (font (size 1.27 1.27)) (justify left))
-    )
-    (property "Value" "130" (id 1) (at 60.96 133.35 90)
-      (effects (font (size 1.27 1.27)) (justify left))
-    )
-    (property "Footprint" "" (id 2) (at 59.182 131.445 90)
-      (effects (font (size 1.27 1.27)) hide)
-    )
-    (property "Datasheet" "~" (id 3) (at 60.96 131.445 0)
-      (effects (font (size 1.27 1.27)) hide)
-    )
-    (pin "1")
-    (pin "2")
-  )
-  (symbol (lib_id "Device:R") (at 55.245 128.905 0) (unit 1)
-    (in_bom yes) (on_board yes)
-    (property "Reference" "R3" (id 0) (at 57.023 127.7366 0)
-      (effects (font (size 1.27 1.27)) (justify left))
-    )
-    (property "Value" "130" (id 1) (at 55.245 130.81 90)
-      (effects (font (size 1.27 1.27)) (justify left))
-    )
-    (property "Footprint" "" (id 2) (at 53.467 128.905 90)
-      (effects (font (size 1.27 1.27)) hide)
-    )
-    (property "Datasheet" "~" (id 3) (at 55.245 128.905 0)
-      (effects (font (size 1.27 1.27)) hide)
-    )
-    (pin "1")
-    (pin "2")
-  )
-  (symbol (lib_id "Device:LED") (at 55.245 137.795 90) (unit 1)
-    (in_bom yes) (on_board yes)
-    (property "Reference" "D3" (id 0) (at 58.42 137.16 0)
-      (effects (font (size 1.27 1.27)) (justify right))
-    )
-    (property "Value" "Blue" (id 1) (at 58.42 132.715 0)
-      (effects (font (size 1.27 1.27)) (justify right))
-    )
-    (property "Footprint" "" (id 2) (at 55.245 137.795 0)
-      (effects (font (size 1.27 1.27)) hide)
-    )
-    (property "Datasheet" "~" (id 3) (at 55.245 137.795 0)
-      (effects (font (size 1.27 1.27)) hide)
-    )
-    (pin "1")
-    (pin "2")
-  )
-  (symbol (lib_id "Device:LED") (at 66.675 151.765 90) (unit 1)
-    (in_bom yes) (on_board yes)
-    (property "Reference" "D5" (id 0) (at 69.85 151.13 0)
-      (effects (font (size 1.27 1.27)) (justify right))
-    )
-    (property "Value" "Blue" (id 1) (at 69.85 146.685 0)
-      (effects (font (size 1.27 1.27)) (justify right))
-    )
-    (property "Footprint" "" (id 2) (at 66.675 151.765 0)
-      (effects (font (size 1.27 1.27)) hide)
-    )
-    (property "Datasheet" "~" (id 3) (at 66.675 151.765 0)
-      (effects (font (size 1.27 1.27)) hide)
-    )
-    (pin "1")
-    (pin "2")
-  )
-  (symbol (lib_id "Device:LED") (at 60.96 144.78 90) (unit 1)
-    (in_bom yes) (on_board yes)
-    (property "Reference" "D4" (id 0) (at 64.135 144.145 0)
-      (effects (font (size 1.27 1.27)) (justify right))
-    )
-    (property "Value" "Blue" (id 1) (at 64.135 139.7 0)
-      (effects (font (size 1.27 1.27)) (justify right))
-    )
-    (property "Footprint" "" (id 2) (at 60.96 144.78 0)
-      (effects (font (size 1.27 1.27)) hide)
-    )
-    (property "Datasheet" "~" (id 3) (at 60.96 144.78 0)
-      (effects (font (size 1.27 1.27)) hide)
-    )
-    (pin "1")
-    (pin "2")
-  )
-  (symbol (lib_id "power:GND") (at 66.675 157.48 0) (unit 1)
-    (in_bom yes) (on_board yes)
-    (property "Reference" "#PWR039" (id 0) (at 66.675 163.83 0)
-      (effects (font (size 1.27 1.27)) hide)
-    )
-    (property "Value" "GND" (id 1) (at 66.802 161.8742 0))
-    (property "Footprint" "" (id 2) (at 66.675 157.48 0)
-      (effects (font (size 1.27 1.27)) hide)
-    )
-    (property "Datasheet" "" (id 3) (at 66.675 157.48 0)
-      (effects (font (size 1.27 1.27)) hide)
-    )
-    (pin "1")
-  )
-  (symbol (lib_id "power:GND") (at 60.96 150.495 0) (unit 1)
-    (in_bom yes) (on_board yes)
-    (property "Reference" "#PWR038" (id 0) (at 60.96 156.845 0)
-      (effects (font (size 1.27 1.27)) hide)
-    )
-    (property "Value" "GND" (id 1) (at 61.087 154.8892 0))
-    (property "Footprint" "" (id 2) (at 60.96 150.495 0)
-      (effects (font (size 1.27 1.27)) hide)
-    )
-    (property "Datasheet" "" (id 3) (at 60.96 150.495 0)
-      (effects (font (size 1.27 1.27)) hide)
-    )
-    (pin "1")
-  )
-  (symbol (lib_id "power:GND") (at 55.245 143.51 0) (unit 1)
-    (in_bom yes) (on_board yes)
-    (property "Reference" "#PWR037" (id 0) (at 55.245 149.86 0)
-      (effects (font (size 1.27 1.27)) hide)
-    )
-    (property "Value" "GND" (id 1) (at 55.372 147.9042 0))
-    (property "Footprint" "" (id 2) (at 55.245 143.51 0)
-      (effects (font (size 1.27 1.27)) hide)
-    )
-    (property "Datasheet" "" (id 3) (at 55.245 143.51 0)
-      (effects (font (size 1.27 1.27)) hide)
-    )
-    (pin "1")
-  )
   (symbol (lib_id "Connector:RJ45_LED_Shielded") (at 189.865 52.705 270) (unit 1)
