File: Hardware/ScienceSensor/ScienceSensor.kicad_sch (KiCad schematic)
At the start: 15 parts, among them U1 OKI-78SR-5_1.5-W36H-C, U2 OKI-78SR-3.3_1.5-W36H-C

Commit message: Schematic Review
Parts:
- removed C1: CP1, symbol ScienceSensor-rescue:CP1-Device
- removed C3: 10uF, symbol Device:C
- removed U1: OKI-78SR-5_1.5-W36H-C, Converter_DCDC:Converter_DCDC_muRata_OKI-78SR_Horizontal, symbol Converter_DCDC:OKI-78SR-5_1.5-W36H-C
- added U?: TSR_1-2450, Converter_DCDC:Converter_DCDC_TRACO_TSR-1_THT, symbol Regulator_Switching:TSR_1-2450
- R1: value 43 -> 500
Connections:
- net +12V: now also U?.1 (Vin)
- net +5V: now also U?.3 (Vout)
- net GND: now also U?.2 (GND)

Commit message: Hierarchal sheets removed, laser control mosfets moved low-side
Parts:
- added C? (x2): 2.2uF, Capacitor_SMD:C_0603_1608Metric_Pad1.08x0.95mm_HandSolder, symbol Device:C
- added C? (x2): 3.3nF, Capacitor_SMD:C_0603_1608Metric_Pad1.08x0.95mm_HandSolder, symbol Device:C
- added C?: 0.1uF, symbol Device:C
- added Conn? (x3): Molex_SL_02, symbol MRDT_Connectors:Molex_SL_02
- added Conn? (x3): Molex_SL_03, symbol MRDT_Connectors:Molex_SL_03
- added Conn? (x2): Molex_SL_04, symbol MRDT_Connectors:Molex_SL_04
- added Conn?: Molex_SL_05, MRDT_Connectors:MOLEX_SL_05_Horizontal, symbol MRDT_Connectors:Molex_SL_05
- added Conn?: Molex_SL_04, MRDT_Connectors:MOLEX_SL_04_Horizontal, symbol MRDT_Connectors:Molex_SL_04
- added D? (x7): Blue, symbol Device:LED
- added J?: RJ45_LED_Shielded, symbol Connector:RJ45_LED_Shielded
- added J?: 6P6C, symbol Connector:6P6C
- added Q? (x3): BSS214NW, Package_TO_SOT_SMD:SOT-323_SC-70, symbol Transistor_FET:BSS214NW
- added Q? (x7): BSS138, symbol Device:Q_NMOS_GSD
- added R? (x14): 10K, symbol Device:R
- added R? (x3): 100, symbol Device:R
- added R? (x4): 500, symbol Device:R
- added R? (x2): 1M, Resistor_SMD:R_0603_1608Metric_Pad0.98x0.95mm_HandSolder, symbol Device:R
- added R? (x2): 56k, Resistor_SMD:R_0603_1608Metric_Pad0.98x0.95mm_HandSolder, symbol Device:R
- added U?: Teensy4.1_DEV-16771, MODULE_DEV-16771, symbol MRDT_Shields:Teensy4.1_DEV-16771
- added U? (x2): TSV911RILT, Package_TO_SOT_SMD:SOT-23-5, symbol Amplifier_Operational:TSV911RILT
Connections:
- net +12V: now also Conn?.1, Conn?.1, Conn?.1
- net +3V3: now also Q?.1 (G), Q?.1 (G), Q?.1 (G), Q?.1 (G), Q?.1 (G), Q?.1 (G), Q?.1 (G), R?.1, R?.1, R?.1, R?.1, R?.1, R?.1, R?.1, U?.3.3V_1 (3.3V), U?.3.3V_2 (3.3V), U?.3.3V_3 (3.3V)
- net +5V: now also Conn?.1, Conn?.1, Conn?.1, Conn?.1, R?.1, R?.1, R?.1, R?.1, R?.1, R?.1, R?.1, U?.2 (V+), U?.2 (V+), U?.5V
- net GND: now also C?.2, C?.2, Conn?.2, Conn?.2, Conn?.2, Conn?.2, Conn?.2, Conn?.2, Conn?.2, D?.1 (K), D?.1 (K), D?.1 (K), D?.1 (K), D?.1 (K), D?.1 (K), D?.1 (K), J?.SH, Q?.2 (S), Q?.2 (S), Q?.2 (S), U?.5 (V-), U?.5 (V-), U?.GND1 (GND), U?.GND2 (GND), U?.GND3 (GND), U?.GND4 (GND), U?.GND5 (GND)
- new net: Conn?.2, Q?.3 (D) (x3)
- new net: D?.2 (A), R?.1 (x7)
- new net: C?.1, R?.2 (x2)
- new net: U?.USB_GND1 (USB_GND), U?.USB_GND2 (USB_GND)
- new net: J?.1, J?.1
- new net: J?.10, J?.4
- new net: C?.1, J?.2, J?.5
- new net: J?.2, J?.3
- new net: J?.4, J?.6
- new net: J?.5, J?.6
- new net: C?.2, J?.3, J?.8, J?.9
- new net: C?.1, R?.1, R?.1, U?.4 (-) (x2)
- new net: Conn?.4, U?.3 (+)
- new net: Conn?.3, U?.3 (+)
- new net +3.3V: Conn?.1, Conn?.1, Conn?.1
- new net CO2_RX: Conn?.4, Q?.3 (D), R?.2, R?.2
- new net CO2_TX: Conn?.3, Q?.3 (D), R?.2, R?.2
- new net Laser_1: Q?.1 (G), R?.2, U?.14 (A0)
- new net Laser_2: Q?.1 (G), R?.2, U?.15 (A1)
- new net Laser_3: Q?.1 (G), R?.2, U?.16 (A2)
- new net Lights: U?.19 (A5)
- new net NO2_CS: Conn?.4, Q?.3 (D), R?.2
- new net NO2_MISO: Conn?.3, Q?.3 (D), R?.2
- new net NO2_SCK: Conn?.5, Q?.3 (D), R?.2
- new net NO_Gas: C?.2, R?.2, U?.1, U?.41 (A17)
- new net NO_Ref: C?.2, R?.2, U?.1, U?.40 (A16)
- new net O2_RX: Conn?.4, Q?.3 (D), R?.2, R?.2
- new net O2_TX: Conn?.3, Q?.3 (D), R?.2, R?.2
- new net Photodiode_1: Conn?.3, U?.25 (A11)
- new net Photodiode_2: Conn?.3, U?.24 (A10)
- new net Photodiode_3: Conn?.3, U?.23 (A9)
- new net Teensy_CO2_RX: Q?.2 (S), R?.2, U?.7 (RX2)
- new net Teensy_CO2_TX: Q?.2 (S), R?.2, U?.8 (TX2)
- new net Teensy_NO2_CS: Q?.2 (S), R?.2, U?.10 (CS1)
- new net Teensy_NO2_MISO: Q?.2 (S), R?.2, U?.12 (MISO)
- new net Teensy_NO2_SCK: Q?.2 (S), R?.2, U?.13 (SCK)
- new net Teensy_O2_RX: Q?.2 (S), R?.2, U?.0 (RX1)
- new net Teensy_O2_TX: Q?.2 (S), R?.2, U?.1 (TX1)
- new net UV_Lights: U?.18 (A4)
- no-connect marks 0 -> 41
Other:
- removed sheet Lasers & Photodiode
- removed sheet Sensors
- removed sheet Teensy
- note added: "CO2_Sensor"
- note added: "Laser 1"
- note added: "Laser 2"
- note added: "Laser 3"
- note added: "MOSFETS"
- note added: "NO2_Sensor"
- note added: "NO_Sensor"
- note added: "O2_Sensor"
- note added: "Photodiode 1"
- note added: "Photodiode 2"
- note added: "Photodiode 3"
- moved on the sheet: C2, C4, Conn1A, Conn1B, D1, D2, R1, R2, U2, U?, V1, V2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
