File: Hardware/ScienceSensorBoard/ScienceSensor.kicad_pcb (KiCad board)
At the start: 2 copper layers, 96.5 x 94.5 mm, 70 parts, among them J1 RJ45_LED_Shielded, J2 Conn_02x03_Counter_Clockwise, Q1 BSS138, Q2 BSS138, Q3 BSS138, Q4 BSS138, Q5 BSS138, Q6 BSS138, Q7 BSS138, U1 TSR_1-2450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

Commit message: Changed teensy footprint
Parts:
- U2: footprint MRDT_Shields:Teensy_4_1 -> MRDT_Shields:Teensy_4_1_Bare
Routing:
- net +5V: track 324.2 -> 309.4 mm
- net +3V3: track 391.9 -> 390.4 mm

Commit message: Generated BOM + Gerbs
Routing:
- net Teensy_O2_TX: track 41.7 -> 38.2 mm
- net Teensy_O2_RX: track 37.3 -> 34.1 mm
- net Net-(C1-Pad2): track 32.0 -> 33.6 mm
- net GND: vias 40 -> 41
Changed lines of the file:
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@@
       (layerselection 0x00010fc_ffffffff)
       (disableapertmacros false)
-      (usegerberextensions false)
+      (usegerberextensions true)
       (usegerberattributes true)
-      (usegerberadvancedattributes true)
-      (creategerberjobfile true)
+      (usegerberadvancedattributes false)
+      (creategerberjobfile false)
       (svguseinch false)
       (svgprecision 6)
@@
       (psa4output false)
       (plotreference true)
-      (plotvalue true)
+      (plotvalue false)
       (plotinvisibletext false)
       (sketchpadsonfab false)
-      (subtractmaskfromsilk false)
+      (subtractmaskfromsilk true)
       (outputformat 1)
       (mirror false)
-      (drillshape 1)
+      (drillshape 0)
       (scaleselection 1)
-      (outputdirectory "")
+      (outputdirectory "../../Documentation/Main Board Gerbs/")
     )
   )
@@
     (fp_line (start -2.5 1.79) (end -2.5 2.55) (layer "F.Fab") (width 0.1))
     (fp_line (start 2.54 4.05) (end 10.16 4.05) (layer "F.Fab") (width 0.1))
-    (pad "1" thru_hole roundrect (at 0 0 270) (size 1.74 1.74) (drill 1.09) (layers *.Cu *.Mask) (roundrect_rratio 0.143678)
+    (pad "1" thru_hole roundrect (at 0 0 270) (size 1.74 1.74) (drill 1.09) (layers *.Cu *.Mask) (roundrect_rratio 0.1436781609)
       (net 5 "+3V3") (pintype "input"))
     (pad "2" thru_hole circle (at 2.54 0 270) (size 1.74 1.74) (drill 1.09) (layers *.Cu *.Mask)
@@
     (fp_line (start -2.5 2.55) (end 15.2 2.55) (layer "F.Fab") (width 0.1))
     (fp_line (start 0.5 -2.55) (end 0 -1.842893) (layer "F.Fab") (width 0.1))
-    (pad "1" thru_hole roundrect (at 0 0 270) (size 1.74 1.74) (drill 1.09) (layers *.Cu *.Mask) (roundrect_rratio 0.143678)
+    (pad "1" thru_hole roundrect (at 0 0 270) (size 1.74 1.74) (drill 1.09) (layers *.Cu *.Mask) (roundrect_rratio 0.1436781609)
       (net 3 "+12V") (pintype "input"))
     (pad "2" thru_hole circle (at 2.54 0 270) (size 1.74 1.74) (drill 1.09) (layers *.Cu *.Mask)
@@
   )
   (segment (start 175.514 64.006) (end 175.514 65.276) (width 0.254) (layer "F.Cu") (net 1))
-  (segment (start 171.31 61.859) (end 173.367 61.859) (width 0.254) (layer "F.Cu") (net 1))
-  (segment (start 167.996 58.545) (end 171.31 61.859) (width 0.254) (layer "F.Cu") (net 1))
-  (segment (start 173.367 61.859) (end 175.514 64.006) (width 0.254) (layer "F.Cu") (net 1))
+  (segment (start 170.942 61.468) (end 170.9305 61.4795) (width 0.254) (layer "F.Cu") (net 1))
+  (segment (start 175.514 64.006) (end 175.514 63.246) (width 0.254) (layer "F.Cu") (net 1))
+  (segment (start 170.9305 61.4795) (end 167.996 58.545) (width 0.254) (layer "F.Cu") (net 1))
+  (segment (start 173.736 61.468) (end 170.942 61.468) (width 0.254) (layer "F.Cu") (net 1))
   (segment (start 175.514 65.276) (end 172.974 67.816) (width 0.254) (layer "F.Cu") (net 1))
+  (segment (start 175.514 63.246) (end 173.736 61.468) (width 0.254) (layer "F.Cu") (net 1))
   (segment (start 171.323 58.545) (end 172.974 60.196) (width 0.254) (layer "F.Cu") (net 2))
   (segment (start 169.721 58.545) (end 171.323 58.545) (width 0.254) (layer "F.Cu") (net 2))
-  (segment (start 180.213 67.435) (end 182.3205 67.435) (width 0.254) (layer "F.Cu") (net 2))
-  (segment (start 172.974 60.196) (end 180.213 67.435) (width 0.254) (layer "F.Cu") (net 2))
-  (segment (start 185.8515 70.966) (end 186.944 70.966) (width 0.254) (layer "F.Cu") (net 2))
-  (segment (start 182.3205 67.435) (end 185.8515 70.966) (width 0.254) (layer "F.Cu") (net 2))
+  (segment (start 172.974 60.196) (end 178.814 60.196) (width 0.254) (layer "F.Cu") (net 2))
+  (segment (start 186.944 68.326) (end 186.944 70.966) (width 0.254) (layer "F.Cu") (net 2))
+  (segment (start 178.814 60.196) (end 186.944 68.326) (width 0.254) (layer "F.Cu") (net 2))
   (segment (start 172.974 60.196) (end 172.097 61.073) (width 0.254) (layer "B.Cu") (net 2))
   (segment (start 172.097 61.073) (end 172.097 66.393) (width 0.254) (layer "B.Cu") (net 2))
@@
   (via (at 181.102 116.84) (size 0.8) (drill 0.4) (layers "F.Cu" "B.Cu") (free) (net 4))
   (via (at 177.8 109.982) (size 0.8) (drill 0.4) (layers "F.Cu" "B.Cu") (free) (net 4))
+  (via (at 154.94 94.996) (size 0.8) (drill 0.4) (layers "F.Cu" "B.Cu") (free) (net 4))
   (via (at 162.814 69.088) (size 0.8) (drill 0.4) (layers "F.Cu" "B.Cu") (free) (net 4))
   (via (at 135.128 109.22) (size 0.8) (drill 0.4) (layers "F.Cu" "B.Cu") (free) (net 4))
@@
   (via (at 116.586 125.984) (size 0.8) (drill 0.4) (layers "F.Cu" "B.Cu") (free) (net 4))
   (via (at 162.56 76.2) (size 0.8) (drill 0.4) (layers "F.Cu" "B.Cu") (free) (net 4))
-  (via (at 154.94 89.408) (size 0.8) (drill 0.4) (layers "F.Cu" "B.Cu") (free) (net 4))
   (via (at 177.8 84.836) (size 0.8) (drill 0.4) (layers "F.Cu" "B.Cu") (free) (net 4))
   (via (at 154.94 76.2) (size 0.8) (drill 0.4) (layers "F.Cu" "B.Cu") (free) (net 4))
@@
   (via (at 108.204 67.818) (size 0.8) (drill 0.4) (layers "F.Cu" "B.Cu") (free) (net 4))
   (via (at 165.862 89.408) (size 0.8) (drill 0.4) (layers "F.Cu" "B.Cu") (free) (net 4))
+  (via (at 138.43 63.754) (size 0.8) (drill 0.4) (layers "F.Cu" "B.Cu") (free) (net 4))
   (via (at 134.62 94.488) (size 0.8) (drill 0.4) (layers "F.Cu" "B.Cu") (free) (net 4))
   (via (at 162.56 84.836) (size 0.8) (drill 0.4) (layers "F.Cu" "B.Cu") (free) (net 4))
@@
   (segment (start 141.5815 114.427) (end 141.5815 112.9265) (width 0.254) (layer "F.Cu") (net 54))
   (via (at 141.605 112.903) (size 0.8) (drill 0.4) (layers "F.Cu" "B.Cu") (net 54))
-  (segment (start 148.209 99.314) (end 151.765 95.758) (width 0.254) (layer "B.Cu") (net 54))
-  (segment (start 151.765 86.614) (end 152.781 85.598) (width 0.254) (layer "B.Cu") (net 54))
-  (segment (start 152.781 85.598) (end 158.75 85.598) (width 0.254) (layer "B.Cu") (net 54))
-  (segment (start 151.765 95.758) (end 151.765 86.614) (width 0.254) (layer "B.Cu") (net 54))
-  (segment (start 148.209 106.299) (end 148.209 99.314) (width 0.254) (layer "B.Cu") (net 54))
-  (segment (start 141.605 112.903) (end 148.209 106.299) (width 0.254) (layer "B.Cu") (net 54))
+  (segment (start 145.161 109.347) (end 141.605 112.903) (width 0.254) (layer "B.Cu") (net 54))
+  (segment (start 158.75 85.598) (end 145.161 99.187) (width 0.254) (layer "B.Cu") (net 54))
+  (segment (start 145.161 99.187) (end 145.161 109.347) (width 0.254) (layer "B.Cu") (net 54))
   (segment (start 155.26 114.3375) (end 155.2975 114.3) (width 0.254) (layer "F.Cu") (net 55))
   (segment (start 155.321 114.2765) (end 155.2975 114.3) (width 0.254) (layer "F.Cu") (net 55))
@@
   (segment (start 145.3915 112.9265) (end 145.415 112.903) (width 0.254) (layer "F.Cu") (net 58))
   (via (at 145.415 112.903) (size 0.8) (drill 0.4) (layers "F.Cu" "B.Cu") (net 58))
-  (segment (start 152.273 89.154) (end 153.289 88.138) (width 0.254) (layer "B.Cu") (net 58))
-  (segment (start 148.717 109.601) (end 148.717 99.568) (width 0.254) (layer "B.Cu") (net 58))
-  (segment (start 152.273 96.012) (end 152.273 89.154) (width 0.254) (layer "B.Cu") (net 58))
-  (segment (start 148.717 99.568) (end 152.273 96.012) (width 0.254) (layer "B.Cu") (net 58))
-  (segment (start 153.289 88.138) (end 158.75 88.138) (width 0.254) (layer "B.Cu") (net 58))
-  (segment (start 145.415 112.903) (end 148.717 109.601) (width 0.254) (layer "B.Cu") (net 58))
+  (segment (start 145.923 112.395) (end 145.415 112.903) (width 0.254) (layer "B.Cu") (net 58))
+  (segment (start 145.923 100.965) (end 145.923 112.395) (width 0.254) (layer "B.Cu") (net 58))
+  (segment (start 158.75 88.138) (end 145.923 100.965) (width 0.254) (layer "B.Cu") (net 58))
   (segment (start 159.3615 113.8955) (end 159.3615 114.3) (width 0.254) (layer "F.Cu") (net 59))
   (segment (start 159.324 116.5375) (end 159.324 114.3375) (width 0.254) (layer "F.Cu") (net 59))
