File: Hardware/TCD1304AP Breakout/FluorometerDetector (1)/FluorometerDetector (1).kicad_sch (KiCad schematic)
At the start: 10 parts, among them Q1 Q_PNP_BCE, U1 TCD1304

Commit message: missed autosave changes
Parts:
- added C1: 10uF, Capacitor_SMD:C_0603_1608Metric_Pad1.08x0.95mm_HandSolder, symbol Device:C
- added R1: 1.2k, Resistor_SMD:R_0603_1608Metric_Pad0.98x0.95mm_HandSolder, symbol Device:R
- Q1: footprint (none) -> Package_TO_SOT_THT:TO-92_HandSolder; symbol Device:Q_PNP_BCE -> Device:Q_PNP_ECB
- R2: renamed from R1; value 2.2k -> 1k; footprint (none) -> Resistor_SMD:R_0603_1608Metric_Pad0.98x0.95mm_HandSolder
- R3: renamed from R2; footprint (none) -> Resistor_SMD:R_0603_1608Metric_Pad0.98x0.95mm_HandSolder
- R4: renamed from R3; footprint (none) -> Resistor_SMD:R_0603_1608Metric_Pad0.98x0.95mm_HandSolder
Connections:
- net +3V3: now also C1.2, R1.1; no longer R2.1
- net GND: now also C1.1
- net at Conn1.6, R2.2: now also Q1.1 (E); no longer Q1.3 (E)
- net at R3.2: now also Q1.3 (B); no longer Q1.1 (B)
- new net: R1.2, R2.1
Changed lines of the file:
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@@
 (kicad_sch (version 20211123) (generator eeschema)
   (paper "A4")
+  (junction (at 171.45 20.32) (diameter 0) (color 0 0 0 0)
+  )
   (junction (at 130.81 64.77) (diameter 0) (color 0 0 0 0)
   )
   (junction (at 169.545 31.115) (diameter 0) (color 0 0 0 0)
   )
+  (junction (at 171.45 31.115) (diameter 0) (color 0 0 0 0)
+  )
+  (wire (pts (xy 176.53 27.94) (xy 176.53 31.115))
+    (stroke (width 0) (type default) (color 0 0 0 0))
+  )
   (wire (pts (xy 177.8 35.56) (xy 177.8 32.385))
     (stroke (width 0) (type default) (color 0 0 0 0))
@@
     (stroke (width 0) (type default) (color 0 0 0 0))
   )
+  (wire (pts (xy 116.205 64.77) (xy 118.11 64.77))
+    (stroke (width 0) (type default) (color 0 0 0 0))
+  )
   (wire (pts (xy 149.86 29.845) (xy 149.86 40.64))
     (stroke (width 0) (type default) (color 0 0 0 0))
@@
     (stroke (width 0) (type default) (color 0 0 0 0))
   )
-  (wire (pts (xy 115.57 60.96) (xy 115.57 64.77))
+  (wire (pts (xy 108.585 60.325) (xy 108.585 64.77))
     (stroke (width 0) (type default) (color 0 0 0 0))
   )
@@
     (stroke (width 0) (type default) (color 0 0 0 0))
   )
-  (wire (pts (xy 118.11 64.77) (xy 115.57 64.77))
-    (stroke (width 0) (type default) (color 0 0 0 0))
-  )
   (wire (pts (xy 169.545 31.115) (xy 171.45 31.115))
     (stroke (width 0) (type default) (color 0 0 0 0))
@@
     (stroke (width 0) (type default) (color 0 0 0 0))
   )
+  (wire (pts (xy 171.45 31.115) (xy 176.53 31.115))
+    (stroke (width 0) (type default) (color 0 0 0 0))
+  )
   (wire (pts (xy 184.785 43.18) (xy 147.32 43.18))
+    (stroke (width 0) (type default) (color 0 0 0 0))
+  )
+  (wire (pts (xy 171.45 20.32) (xy 176.53 20.32))
     (stroke (width 0) (type default) (color 0 0 0 0))
   )
@@
     (effects (font (size 4 4)) (justify left bottom))
   )
-  (symbol (lib_id "power:+3V3") (at 115.57 60.96 0) (unit 1)
-    (in_bom yes) (on_board yes) (fields_autoplaced)
-    (property "Reference" "#PWR01" (id 0) (at 115.57 64.77 0)
-      (effects (font (size 1.27 1.27)) hide)
-    )
-    (property "Value" "+3V3" (id 1) (at 115.57 57.3842 0))
-    (property "Footprint" "" (id 2) (at 115.57 60.96 0)
-      (effects (font (size 1.27 1.27)) hide)
-    )
-    (property "Datasheet" "" (id 3) (at 115.57 60.96 0)
+  (symbol (lib_id "power:+3V3") (at 108.585 60.325 0) (unit 1)
+    (in_bom yes) (on_board yes) (fields_autoplaced)
+    (property "Reference" "#PWR01" (id 0) (at 108.585 64.135 0)
+      (effects (font (size 1.27 1.27)) hide)
+    )
+    (property "Value" "+3V3" (id 1) (at 108.585 56.7492 0))
+    (property "Footprint" "" (id 2) (at 108.585 60.325 0)
+      (effects (font (size 1.27 1.27)) hide)
+    )
+    (property "Datasheet" "" (id 3) (at 108.585 60.325 0)
       (effects (font (size 1.27 1.27)) hide)
     )
@@
     (pin "1")
   )
+  (symbol (lib_id "Device:R") (at 112.395 64.77 90) (unit 1)
+    (in_bom yes) (on_board yes)
+    (property "Reference" "R1" (id 0) (at 112.395 62.23 90))
+    (property "Value" "1.2k" (id 1) (at 112.395 64.77 90))
+    (property "Footprint" "Resistor_SMD:R_0603_1608Metric_Pad0.98x0.95mm_HandSolder" (id 2) (at 112.395 66.548 90)
+      (effects (font (size 1.27 1.27)) hide)
+    )
+    (property "Datasheet" "~" (id 3) (at 112.395 64.77 0)
+      (effects (font (size 1.27 1.27)) hide)
+    )
+    (pin "1")
+    (pin "2")
+  )
   (symbol (lib_id "power:GND") (at 165.1 66.675 0) (unit 1)
     (in_bom yes) (on_board yes) (fields_autoplaced)
@@
     (pin "1")
   )
+  (symbol (lib_id "Device:C") (at 176.53 24.13 0) (unit 1)
+    (in_bom yes) (on_board yes) (fields_autoplaced)
+    (property "Reference" "C1" (id 0) (at 179.451 23.2953 0)
+      (effects (font (size 1.27 1.27)) (justify left))
+    )
+    (property "Value" "10uF" (id 1) (at 179.451 25.8322 0)
+      (effects (font (size 1.27 1.27)) (justify left))
+    )
+    (property "Footprint" "Capacitor_SMD:C_0603_1608Metric_Pad1.08x0.95mm_HandSolder" (id 2) (at 177.4952 27.94 0)
+      (effects (font (size 1.27 1.27)) hide)
+    )
+    (property "Datasheet" "~" (id 3) (at 176.53 24.13 0)
+      (effects (font (size 1.27 1.27)) hide)
+    )
+    (pin "1")
+    (pin "2")
+  )
   (symbol (lib_id "power:+3V3") (at 171.45 31.115 0) (unit 1)
     (in_bom yes) (on_board yes) (fields_autoplaced)
@@
   (symbol (lib_id "Device:R") (at 121.92 64.77 90) (unit 1)
     (in_bom yes) (on_board yes)
-    (property "Reference" "R1" (id 0) (at 121.92 62.23 90))
-    (property "Value" "2.2k" (id 1) (at 121.92 64.77 90))
-    (property "Footprint" "" (id 2) (at 121.92 66.548 90)
+    (property "Reference" "R2" (id 0) (at 121.92 62.23 90))
+    (property "Value" "1k" (id 1) (at 121.92 64.77 90))
+    (property "Footprint" "Resistor_SMD:R_0603_1608Metric_Pad0.98x0.95mm_HandSolder" (id 2) (at 121.92 66.548 90)
       (effects (font (size 1.27 1.27)) hide)
     )
@@
   (symbol (lib_id "Device:R") (at 139.7 49.53 0) (unit 1)
     (in_bom yes) (on_board yes)
-    (property "Reference" "R2" (id 0) (at 141.478 48.6953 0)
+    (property "Reference" "R3" (id 0) (at 141.478 48.6953 0)
       (effects (font (size 1.27 1.27)) (justify left))
     )
@@
       (effects (font (size 1.27 1.27)) (justify left))
     )
-    (property "Footprint" "" (id 2) (at 137.922 49.53 90)
+    (property "Footprint" "Resistor_SMD:R_0603_1608Metric_Pad0.98x0.95mm_HandSolder" (id 2) (at 137.922 49.53 90)
       (effects (font (size 1.27 1.27)) hide)
     )
@@
   (symbol (lib_id "Device:R") (at 153.67 64.77 90) (unit 1)
     (in_bom yes) (on_board yes)
-    (property "Reference" "R3" (id 0) (at 153.67 62.23 90))
+    (property "Reference" "R4" (id 0) (at 153.67 62.23 90))
     (property "Value" "150" (id 1) (at 153.67 64.77 90))
-    (property "Footprint" "" (id 2) (at 153.67 66.548 90)
+    (property "Footprint" "Resistor_SMD:R_0603_1608Metric_Pad0.98x0.95mm_HandSolder" (id 2) (at 153.67 66.548 90)
       (effects (font (size 1.27 1.27)) hide)
     )
@@
     (pin "2")
   )
-  (symbol (lib_id "Device:Q_PNP_BCE") (at 139.7 62.23 270) (unit 1)
+  (symbol (lib_id "Device:Q_PNP_ECB") (at 139.7 62.23 270) (unit 1)
     (in_bom yes) (on_board yes) (fields_autoplaced)
     (property "Reference" "Q1" (id 0) (at 139.7 68.3498 90))
     (property "Value" "Q_PNP_BCE" (id 1) (at 139.7 70.8867 90))
-    (property "Footprint" "" (id 2) (at 142.24 67.31 0)
+    (property "Footprint" "Package_TO_SOT_THT:TO-92_HandSolder" (id 2) (at 142.24 67.31 0)
       (effects (font (size 1.27 1.27)) hide)
     )
@@
       (reference "#PWR06") (unit 1) (value "+3V3") (footprint "")
     )
+    (path "/3c6bcc61-d095-4839-91e2-046921707796"
+      (reference "C1") (unit 1) (value "10uF") (footprint "Capacitor_SMD:C_0603_1608Metric_Pad1.08x0.95mm_HandSolder")
+    )
     (path "/fa5d2e23-cb22-43d6-9b2d-b288e81d34e5"
       (reference "Conn1") (unit 1) (value "Molex_SL_06") (footprint "UVLEDs:705550040")
     )
     (path "/b0e93359-de99-4c71-ac67-db20d611c11c"
-      (reference "Q1") (unit 1) (value "Q_PNP_BCE") (footprint "")
+      (reference "Q1") (unit 1) (value "Q_PNP_BCE") (footprint "Package_TO_SOT_THT:TO-92_HandSolder")
+    )
+    (path "/20c3997f-a880-4703-a101-975f605b5a7a"
+      (reference "R1") (unit 1) (value "1.2k") (footprint "Resistor_SMD:R_0603_1608Metric_Pad0.98x0.95mm_HandSolder")
     )
     (path "/61832704-2bff-4f44-a800-6bbaa7131809"
-      (reference "R1") (unit 1) (value "2.2k") (footprint "")
+      (reference "R2") (unit 1) (value "1k") (footprint "Resistor_SMD:R_0603_1608Metric_Pad0.98x0.95mm_HandSolder")
     )
     (path "/6a549ebc-0bd7-4aa3-acd3-5012f87e0a6b"
-      (reference "R2") (unit 1) (value "150") (footprint "")
+      (reference "R3") (unit 1) (value "150") (footprint "Resistor_SMD:R_0603_1608Metric_Pad0.98x0.95mm_HandSolder")
     )
     (path "/a4177187-9a75-41e9-8f6d-e8a0e9b3a2dd"
-      (reference "R3") (unit 1) (value "150") (footprint "")
+      (reference "R4") (unit 1) (value "150") (footprint "Resistor_SMD:R_0603_1608Metric_Pad0.98x0.95mm_HandSolder")
     )
     (path "/7b7d6c50-0f51-4d1e-926c-e78a7fc8517e"
